File: hubs/hub-standard/hub-standard.kicad_pcb (KiCad board)
At the start: 4 copper layers, 98 x 72 mm, 57 parts, among them J1 5VSB_IN, J2 PORT1, J3 PORT2, J4 PORT3, J5 PORT4, J6 USB-C, M1 M3 Mount, M2 M3 Mount, M3 M3 Mount, M4 M3 Mount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

Commit message: New DRC pass.
Routing:
- net /+5V_HOLD: track 31.1 -> 38.9 mm
- net +5VSB: track 274.5 -> 267.7 mm, vias 13 -> 12
- net +3V3: track 230.0 -> 228.7 mm
Changed lines of the file:
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@@
 	)
 	(segment
-		(start 138.3625 137.45)
-		(end 136.45 137.45)
-		(width 0.5)
-		(layer "F.Cu")
-		(net "+5VSB")
-	)
-	(segment
 		(start 142 117.92)
 		(end 144 119.92)
@@
 	)
 	(segment
-		(start 136.45 137.45)
-		(end 136 137)
-		(width 0.5)
-		(layer "F.Cu")
-		(net "+5VSB")
-	)
-	(segment
 		(start 105.635 115.975)
 		(end 105.635 118.295)
@@
 	)
 	(via
-		(at 136 137)
-		(size 0.6)
-		(drill 0.3)
-		(layers "F.Cu" "B.Cu")
-		(net "+5VSB")
-	)
-	(via
 		(at 117 157)
 		(size 0.6)
@@
 	)
 	(segment
-		(start 134 135)
-		(end 136 137)
-		(width 1)
-		(layer "B.Cu")
-		(net "+5VSB")
-	)
-	(segment
 		(start 97.2325 100.15)
 		(end 112.8325 100.15)
@@
 	)
 	(segment
-		(start 132.5 135)
-		(end 134 135)
-		(width 1)
-		(layer "B.Cu")
-		(net "+5VSB")
-	)
-	(segment
 		(start 138.56 108.95)
 		(end 138.51 109)
@@
 	)
 	(segment
-		(start 76.51 141.49)
-		(end 76.51 141)
-		(width 0.3)
-		(layer "F.Cu")
-		(net "+3V3")
-	)
-	(segment
 		(start 74.5 140.275)
 		(end 74.225 140)
@@
 	)
 	(segment
-		(start 73.98 139.255)
-		(end 73.98 138.5)
-		(width 0.3)
-		(layer "F.Cu")
-		(net "+3V3")
-	)
-	(segment
 		(start 113.51 109)
 		(end 113.51 108.01)
@@
 	)
 	(segment
-		(start 140.272316 136.7)
+		(start 145 136.7)
 		(end 152.7 136.7)
 		(width 0.5)
@@
 	)
 	(segment
+		(start 143.2 138.5)
+		(end 139.4125 138.5)
+		(width 0.5)
+		(layer "F.Cu")
+		(net "/+5V_HOLD")
+	)
+	(segment
+		(start 140.272316 136.7)
+		(end 145 136.7)
+		(width 0.5)
+		(layer "F.Cu")
+		(net "/+5V_HOLD")
+	)
+	(segment
 		(start 141.195 130.08)
 		(end 142.42 130.08)
@@
 	)
 	(segment
+		(start 145 136.7)
+		(end 143.2 138.5)
+		(width 0.5)
+		(layer "F.Cu")
+		(net "/+5V_HOLD")
+	)
+	(segment
 		(start 139.122316 135.55)
 		(end 140.272316 136.7)
@@
 		(width 0.5)
 		(layer "F.Cu")
+		(net "/+5V_HOLD")
+	)
+	(segment
+		(start 139.4125 138.5)
+		(end 138.3625 137.45)
+		(width 0.5)
+		(layer "F.Cu")

Commit message: PCB DRC Checks additional, added test points.
Parts:
- added FID1: Fiducial_1mm_Mask2mm, cec-Fiducial:Fiducial_1mm_Mask2mm, F.Cu at (80.0, 105.5)
- added FID3: Fiducial_1mm_Mask2mm, cec-Fiducial:Fiducial_1mm_Mask2mm, F.Cu at (155.5, 153.0)
- added FID3: Fiducial_1mm_Mask2mm, cec-Fiducial:Fiducial_1mm_Mask2mm, F.Cu at (80.5, 153.0)
- added TP1: 5VSB, cec-TestPoint:TestPoint_Pad_D1.5mm, F.Cu at (136.0, 150.5)
- added TP2: GND, cec-TestPoint:TestPoint_Pad_D1.5mm, F.Cu at (139.5, 150.5)
- added TP3: 3V3, cec-TestPoint:TestPoint_Pad_D1.5mm, F.Cu at (143.0, 150.5)
- added TP4: 5V_HOLD, cec-TestPoint:TestPoint_Pad_D1.5mm, F.Cu at (146.5, 150.5)
- added TP5: BLACKOUT, cec-TestPoint:TestPoint_Pad_D1.5mm, F.Cu at (92.0, 146.0)
- added TP6: USB_VBUS, cec-TestPoint:TestPoint_Pad_D1.5mm, F.Cu at (150.0, 150.5)
Routing:
- net /USB_VBUS: track 90.7 -> 107.5 mm, vias 5 -> 8
- net +5VSB: track 267.7 -> 281.4 mm, vias 12 -> 13
- net /+5V_HOLD: track 38.9 -> 52.2 mm
- net +3V3: track 228.7 -> 238.4 mm
- net /BLACKOUT_SENSE: track 10.3 -> 15.5 mm
- net GND: track 84.2 -> 88.6 mm, vias 40 -> 41
- net /EN: track 73.3 -> 75.5 mm

Commit message: Added ESD and one more decoupler, fixed DRC.
Parts:
- added C13: 100nF, cec-Capacitor_SMD:C_0603_1608Metric, F.Cu at (111.0, 113.5)
- added D6: USBLC6-2SC6, cec-Package_TO_SOT_SMD:SOT-23-6, F.Cu at (100.5, 149.1)
Routing:
- net /USB_VBUS: track 107.5 -> 114.5 mm, vias 8 -> 9
- net +3V3: track 238.4 -> 242.7 mm
- net GND: track 88.6 -> 92.3 mm, vias 41 -> 43
- net /USB_DP: track 32.2 -> 33.0 mm
- net /USB_DM: track 32.8 -> 33.5 mm

Commit message: hub-standard: reconcile front-end docs to as-built; fix duplicate fiducial
Pre-fab review follow-ups (Hub Standard):

- Reconcile the power front-end docs to the as-built board (spec, README,
  CLAUDE.md). The TPS2121 priority mux does inrush limiting via its soft-start
  (C_SS 2.2uF) and source-side reverse-current blocking, so the v1.1 discrete
  1 ohm 1 W inrush resistor and a separate reverse-polarity diode are SUPERSEDED
  and not populated. This completes the v3.2 Section 2.7 fold-in, which the Hub
  Standard table had not cleaned up. No design decision changed.
- D1 (the +5V_HOLD reverse-isolation Schottky) is built as SB120 (1A/20V);
  noted SS14 (1A/40V) as a drop-in higher-margin alternative (both adequate at
  5V). Docs previously named only SS14.
- Rename a duplicate fiducial: the board had two FID3 and no FID2. The
  bottom-left fiducial is now FID2 (FID1/2/3 unique for pick-and-place).
- .kicad_dru: note that the Power-min-width rule now actually fires (the
  netclass patterns were fixed in the prior commit) and the under-width power
  traces it surfaces are the GUI routing/pour punch-list.
- README status refreshed: the PCB is placed and fully routed (was "layout not
  started"); records the pre-fab punch-list (ground refill/pour, 5VSB trunk
  width, CAN edge traces, C1 via-in-pad, D6 GND via, silk).

https://claude.ai/code/session_018vzBBqght166NSh7aJGKHf
Parts:
- renumbered FID3 to FID2
Changed lines of the file:
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@@
 		(descr "Fiducial, circular marking, 1mm bare copper, 2mm soldermask opening (Level A)")
 		(tags "fiducial")
-		(property "Reference" "FID3"
+		(property "Reference" "FID2"
 			(at 0 2.5 0)
 			(layer "F.SilkS")

Commit message: Appease DRC.
Routing:
- net /USB_VBUS: track 114.5 -> 123.5 mm
- net +5VSB: track 281.4 -> 282.3 mm

Commit message: DRC Final Pass.
Routing:
- net /USB_VBUS: track 123.5 -> 122.5 mm
Changed lines of the file:
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@@
 	)
 	(segment
-		(start 155.425 115.024999)
-		(end 163.329999 115.024999)
-		(width 0.5)
+		(start 155.825 115.25)
+		(end 155.8 115.275)
+		(width 1)
 		(layer "F.Cu")
 		(net "/5VSB_RAW")
 	)
 	(segment
-		(start 155.425 115.024999)
-		(end 155.500001 115.1)
-		(width 0.4)
+		(start 155.8 116.925)
+		(end 155.8 115.275)
+		(width 1)
 		(layer "F.Cu")
 		(net "/5VSB_RAW")
 	)
 	(segment
-		(start 155.500001 115.1)
-		(end 155.5 117.225)
-		(width 0.4)
+		(start 163.555 115.25)
+		(end 155.825 115.25)
+		(width 1)
+		(layer "F.Cu")
+		(net "/5VSB_RAW")
+	)
+	(segment
+		(start 155.5 117.225)
+		(end 155.8 116.925)
+		(width 1)
 		(layer "F.Cu")
 		(net "/5VSB_RAW")
@@
 	)
 	(segment
-		(start 97.45 155.05)
-		(end 97.5 155)
+		(start 103 155)
+		(end 102.35 155.65)
 		(width 0.3)
 		(layer "F.Cu")
@@
 	)
 	(segment
-		(start 97.45 157.33)
-		(end 97.45 155.05)
+		(start 97.45 155.95)
+		(end 97 155.5)
 		(width 0.3)
 		(layer "F.Cu")
@@
 	)
 	(segment
-		(start 102.35 157.13)
-		(end 102.55 157.33)
+		(start 100.55 150.275)
+		(end 100.55 151.45)
 		(width 0.3)
 		(layer "F.Cu")
@@
 	)
 	(segment
-		(start 100.55 150.275)
-		(end 100.55 151.45)
+		(start 97.45 157.33)
+		(end 97.45 155.95)
 		(width 0.3)
 		(layer "F.Cu")
@@
 	)
 	(segment
-		(start 102.35 155)
-		(end 102.35 157.13)
-		(width 0.3)
-		(layer "F.Cu")
-		(net "/USB_VBUS")
-	)
-	(segment
 		(start 153.95 115.049999)
 		(end 153.95 115.799998)
@@
 	)
 	(segment
-		(start 102.35 155)
-		(end 103 155)
-		(width 0.5)
-		(layer "F.Cu")
-		(net "/USB_VBUS")
-	)
-	(segment
 		(start 97.5 155)
 		(end 97 155.5)
@@
 		(layer "F.Cu")
 		(net "/USB_VBUS")
+	)
+	(segment
+		(start 102.35 155.65)
+		(end 102.35 157.13)
+		(width 0.3)
+		(layer "F.Cu")
+		(net "/USB_VBUS")

Commit message: 3.5V Regulator Buffer Added and cleared more DRC.
Parts:
- added C14: 100nF, cec-Capacitor_SMD:C_0402_1005Metric, F.Cu at (106.5, 121.5)
- added R14: 330Ω, cec-Resistor_SMD:R_0402_1005Metric, F.Cu at (106.5, 124.0)
- added U6: 74AHCT1G34, cec-Package_TO_SOT_SMD:SOT-23-5, F.Cu at (103.0, 123.0)
- J2, J3, J4, J5: footprint cec-Connector_RJ:RJ45_Amphenol_54602-x08_Horizontal -> cec:RJ45_FTP_Shielded_Horizontal
Connections:
- DL1 pad 3: /LED_DATA -> /LED_DATA_DIN
Routing:
- net /LED_DATA: track 34.6 -> 11.7 mm, vias 2 -> 0
- net /LED_DATA_DIN: track 0.00 -> 14.9 mm
- net +5VSB: track 282.3 -> 290.7 mm
- net GND: track 92.3 -> 96.3 mm, vias 43 -> 45
- net /LED_DATA_BUF: track 0.00 -> 1.87 mm
- net /USB_VBUS: track 122.5 -> 121.8 mm

Commit message: PCB Edits.
Parts:
- added C15: 100nF, cec-Capacitor_SMD:C_0402_1005Metric, F.Cu at (199.1, 125.6)
- added C16: 100nF, cec-Capacitor_SMD:C_0402_1005Metric, F.Cu at (199.1, 127.6)
- added C_SS2: 2.2uF, cec-Capacitor_SMD:C_0603_1608Metric, F.Cu at (195.8, 142.5)
- added D7: PESD5V0S1BA, cec-Diode_SMD:D_SOD-323, F.Cu at (196.0, 139.8)
- added J7: CEC_NANOKVM_AUX_5P, cec-Connector_JST:JST_PH_B5B-PH-K-S_1x05_P2.00mm_Vertical, F.Cu at (187.2, 118.5)
- added J8: MAIN_5V_IN, cec-Connector_JST:JST_XH_S2B-XH-A_1x02_P2.50mm_Horizontal, F.Cu at (183.5, 127.8)
- added R15: 47kΩ, cec-Resistor_SMD:R_0402_1005Metric, F.Cu at (195.3, 131.4)
- added R16: 10kΩ, cec-Resistor_SMD:R_0402_1005Metric, F.Cu at (195.3, 133.4)
- added R17: 47kΩ, cec-Resistor_SMD:R_0402_1005Metric, F.Cu at (195.3, 135.3)
- added R18: 10kΩ, cec-Resistor_SMD:R_0402_1005Metric, F.Cu at (195.3, 137.3)
- added R19: 33Ω, cec-Resistor_SMD:R_0402_1005Metric, F.Cu at (198.2, 131.4)
- added R20: 33Ω, cec-Resistor_SMD:R_0402_1005Metric, F.Cu at (198.2, 133.4)
- added R21: 47kΩ, cec-Resistor_SMD:R_0402_1005Metric, F.Cu at (198.2, 135.3)
- added R22: 10kΩ, cec-Resistor_SMD:R_0402_1005Metric, F.Cu at (198.2, 137.3)
- added R23: 47kΩ, cec-Resistor_SMD:R_0402_1005Metric, F.Cu at (201.1, 131.4)
- added R24: 10kΩ, cec-Resistor_SMD:R_0402_1005Metric, F.Cu at (201.1, 133.4)
- added R25: 10kΩ, cec-Resistor_SMD:R_0402_1005Metric, F.Cu at (201.1, 135.3)
- added R_ILIM2: 27kΩ, cec-Resistor_SMD:R_0402_1005Metric, F.Cu at (201.1, 137.3)
- added TH1: NTC 10k, cec-Resistor_SMD:NTC_0402_1005Metric, F.Cu at (199.6, 143.4)
- added U7: TPS2121RUXR, cec-Package_DFN_QFN:RUX0012A, F.Cu at (199.9, 140.3)
- D1: value SB120 -> SS14
- D2, D3, D4, D5: value PESD5V0S1UL -> PESD5V0S1BA
- R3, R4: value 60Ω -> 60.4
- SW_BOOT: renamed from SW2; footprint cec-Button_Switch_SMD:Panasonic_EVQPUJ_EVQPUA -> cec-Button_Switch_SMD:TS-1088-AR02016
- SW_RESET: renamed from SW1; footprint cec-Button_Switch_SMD:Panasonic_EVQPUJ_EVQPUA -> cec-Button_Switch_SMD:TS-1088-AR02016
- U2: value TJA1462A -> TJA1051T/3
- U6: value 74AHCT1G34 -> SN74AHCT1G08
- renumbered TP3 to TP_3V3, TP1 to TP_5VSB, TP2 to TP_GND, TP6 to TP_VBUS, TP4 to TP_VHOLD
Connections:
- U1 pad 15: unconnected-(U1-IO3-Pad15) -> /TEMP_HUB
- U1 pad 17: unconnected-(U1-IO9-Pad17) -> /MAIN_5V_SENSE
- U1 pad 18: unconnected-(U1-IO10-Pad18) -> /5VSB_SENSE
- U1 pad 19: unconnected-(U1-IO11-Pad19) -> /AUX_UART_TX
- U1 pad 20: unconnected-(U1-IO12-Pad20) -> /AUX_UART_RX
- U1 pad 38: unconnected-(U1-IO2-Pad38) -> /HUB_3V3_SENSE
- U1 pad 39: unconnected-(U1-IO1-Pad39) -> /KVM_3V3_SENSE
- U5 pad 1: +5VSB -> /PSU_5V
- U5 pad 8: +5VSB -> /PSU_5V
- U6 pad 1: unconnected-(U6-NC-Pad1) -> /LED_DATA
Routing:
- net /USB_VBUS: track 121.8 -> 121.3 mm
