File: hubs/hub-enterprise/05a-port6.kicad_sch (KiCad schematic)
At the start: 8 parts

Commit message: Beta lock register: verified locks, a new systemic BOM defect, sharpened decisions
Twelve-agent investigation (six web-enabled investigators, each
adversarially verified live). Locks: hub C1 is the Samxon part already
shipping (the Panasonic reference was documentation-only and is out of
stock); no pegless PCIe-keyed header exists anywhere (45586 stays;
0-stock/9-week fab flag); no cross-vendor sensor drop-ins (INA237 as
TI-internal alternate for the thin INA238 line); power-in consolidation
part = S3B-XH-A with GND-center pin order. The adversarial pass caught
a NEW systemic defect: Manufacturer and LCSC properties are swapped
across nearly the whole sourced BOM on EPS and both PCIe schematics
(whole-board JLC import failure; hub/12VHPWR clean) — fix agent
running; plus the USB-C sourcing line carries the wrong manufacturer's
part (correct: XKB C319148). D-11 gained prior art (a community
JLC-corrected variant of this exact footprint exists — vet before
accepting a DRU exception); the 24-pin incumbent form lost its last
defense (no commodity F-F cable exists anywhere, verified).

Co-Authored-By: Claude Fable 5 <noreply@anthropic.com>
Claude-Session: https://claude.ai/code/session_011q5bmwF5BFtSf8Ft5vT1DZ
Other:
- note added: "VCC: SS110 100V series block + SMAJ58A tail-risk TVS (REQ-HUB-COMMON-110). DETECT: 10k series R [BOM names 1206 pkg, captured as 0402 -- flagged] -> PESD5V0S1BA (LOCKED Sec2.4) + 10k pull-up to +3V3 (Sec2.3 code read). pin-7: 100R series R [illustrative] + SMAJ58A tail-risk clamp (REQ-HUB-COMMON-112/114). All pin-7/DETECT-series values are a schematic-capture/bench-calibration task per hub-ent-bo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"
- note removed: "VCC: SS110 100V series block + SMAJ58A tail-risk TVS (REQ-HUB-COMMON-110); DETECT: 10k series R [BOM names 1206 pkg, captured as 0402 here -- flagged] -> PESD5V0S1BA (LOCKED Sec2.4) + 10k pull-up to +3V3 (Sec2.3 code read); pin-7: 100R series R [illustrative] + SMAJ58A tail-risk clamp (REQ-HUB-COMMON-112/114). All pin-7/DETECT-series values are a schematic-capture/bench-calibration task per hub-e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"
