File: modules/eps-8pin/02-can.kicad_sch (KiCad schematic)
At the start: 6 parts, among them U2 TJA1051T/3

Commit message: Wave-2 EPS finalized: ERC posture + hierarchy-aware audit + driver mutator battery
- name-pin stub ERC: measured KiCad FP class (root local label on {wire,
  sheet-pin} subgraph); root hier labels illegal; erc_exclusions CLASS-LOOSE
  (wrong uuid+position suppressed all 13 - measured) -> driver downgrades
  label_dangling to warning per-board (.kicad_pro, netclasses untouched);
  audit-sch keeps real-dangler teeth (verified). ERC errors 1 vs baseline 2.
- audit-sch.py hierarchy upgrade: per-dir expected instance-path chains
  (root-walked, teeth: bad chain FAILs) + hier/global-label + sheet-pin wire
  anchors -> eps 8/8 ok, ent noise collapsed to its real residuals (FOLLOWUPS).
- driver: project name = .kicad_pro basename (GUI instance-rewrite hazard);
  round-3 mutator battery in-generator (G5 26->7 glyph, identity 58/58 held).
- waivers doc: eps composed-engine floor recorded (1/17/7).

Co-Authored-By: Claude Fable 5 <noreply@anthropic.com>
Claude-Session: https://claude.ai/code/session_01LvfqcnEeuin2oyJQw548EX
Changed lines of the file:
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@@
 		(pin "6")
 		(instances
-			(project "eps-8pin"
+			(project "eps8pin-module"
 				(path "/ef7f6c4c-2dd9-4559-b472-96b33604786a/9b7ee0db-a842-437d-bf22-9658a349fa84" (reference "U2") (unit 1))
 			)
@@
 		(pin "2")
 		(instances
-			(project "eps-8pin"
+			(project "eps8pin-module"
 				(path "/ef7f6c4c-2dd9-4559-b472-96b33604786a/9b7ee0db-a842-437d-bf22-9658a349fa84" (reference "C4") (unit 1))
 			)
@@
 		(pin "2")
 		(instances
-			(project "eps-8pin"
+			(project "eps8pin-module"
 				(path "/ef7f6c4c-2dd9-4559-b472-96b33604786a/9b7ee0db-a842-437d-bf22-9658a349fa84" (reference "C8") (unit 1))
 			)
@@
 		(pin "4")
 		(instances
-			(project "eps-8pin"
+			(project "eps8pin-module"
 				(path "/ef7f6c4c-2dd9-4559-b472-96b33604786a/9b7ee0db-a842-437d-bf22-9658a349fa84" (reference "FL1") (unit 1))
 			)
@@
 		(pin "2")
 		(instances
-			(project "eps-8pin"
+			(project "eps8pin-module"
 				(path "/ef7f6c4c-2dd9-4559-b472-96b33604786a/9b7ee0db-a842-437d-bf22-9658a349fa84" (reference "R11") (unit 1))
 			)
@@
 		(pin "2")
 		(instances
-			(project "eps-8pin"
+			(project "eps8pin-module"
 				(path "/ef7f6c4c-2dd9-4559-b472-96b33604786a/9b7ee0db-a842-437d-bf22-9658a349fa84" (reference "R12") (unit 1))
 			)
@@
 	(wire (pts (xy 201.93 105.41) (xy 201.93 101.6))
 		(stroke (width 0) (type default)))
-	(wire (pts (xy 144.78 91.44) (xy 140.97 91.44))
+	(wire (pts (xy 144.78 91.44) (xy 139.7 91.44))
 		(stroke (width 0) (type default)))
 	(wire (pts (xy 140.97 83.82) (xy 121.92 83.82))
@@
 		(pin "1")
 		(instances
-			(project "eps-8pin"
+			(project "eps8pin-module"
 				(path "/ef7f6c4c-2dd9-4559-b472-96b33604786a/9b7ee0db-a842-437d-bf22-9658a349fa84" (reference "#PWR201") (unit 1))
 			)
@@
 		(pin "1")
 		(instances
-			(project "eps-8pin"
+			(project "eps8pin-module"
 				(path "/ef7f6c4c-2dd9-4559-b472-96b33604786a/9b7ee0db-a842-437d-bf22-9658a349fa84" (reference "#PWR202") (unit 1))
 			)
@@
 		(pin "1")
 		(instances
-			(project "eps-8pin"
+			(project "eps8pin-module"
 				(path "/ef7f6c4c-2dd9-4559-b472-96b33604786a/9b7ee0db-a842-437d-bf22-9658a349fa84" (reference "#PWR203") (unit 1))
 			)
@@
 		(pin "1")
 		(instances
-			(project "eps-8pin"
+			(project "eps8pin-module"
 				(path "/ef7f6c4c-2dd9-4559-b472-96b33604786a/9b7ee0db-a842-437d-bf22-9658a349fa84" (reference "#PWR204") (unit 1))
 			)
@@
 		(pin "1")
 		(instances
-			(project "eps-8pin"
+			(project "eps8pin-module"
 				(path "/ef7f6c4c-2dd9-4559-b472-96b33604786a/9b7ee0db-a842-437d-bf22-9658a349fa84" (reference "#PWR205") (unit 1))
 			)
@@
 		(pin "1")
 		(instances
-			(project "eps-8pin"
+			(project "eps8pin-module"
 				(path "/ef7f6c4c-2dd9-4559-b472-96b33604786a/9b7ee0db-a842-437d-bf22-9658a349fa84" (reference "#PWR206") (unit 1))
 			)
@@
 		(pin "1")
 		(instances
-			(project "eps-8pin"
+			(project "eps8pin-module"
 				(path "/ef7f6c4c-2dd9-4559-b472-96b33604786a/9b7ee0db-a842-437d-bf22-9658a349fa84" (reference "#PWR207") (unit 1))
 			)
@@
 	(symbol
 		(lib_id "cec-power:+3V3")
-		(at 140.97 91.44 180)
-		(unit 1)
-		(exclude_from_sim no)
-		(in_bom yes)
-		(on_board yes)
-		(dnp no)
-		(property "Reference" "#PWR208" (at 140.97 88.9 0) (effects (font (size 1.27 1.27)) (hide yes)))
-		(property "Value" "+3V3" (at 140.97 96.52 0) (effects (font (size 1.27 1.27))))
-		(pin "1")
-		(instances
-			(project "eps-8pin"
+		(at 139.7 91.44 180)
+		(unit 1)
+		(exclude_from_sim no)
+		(in_bom yes)
+		(on_board yes)
+		(dnp no)
+		(property "Reference" "#PWR208" (at 139.7 88.9 0) (effects (font (size 1.27 1.27)) (hide yes)))
+		(property "Value" "+3V3" (at 139.7 96.52 0) (effects (font (size 1.27 1.27))))
+		(pin "1")
+		(instances
+			(project "eps8pin-module"
 				(path "/ef7f6c4c-2dd9-4559-b472-96b33604786a/9b7ee0db-a842-437d-bf22-9658a349fa84" (reference "#PWR208") (unit 1))
 			)
