File: modules/atx-24pin-rev3/24pin-module.kicad_sch (KiCad schematic)
At the start: 74 parts, among them J1 TO-HUB, J2 TO-HUB-PWR, J3 ATX-24 PSU, J5 USB-C 2.0, J6 TO-HUB-STACK, SW1 BOOT, SW2 RESET, U1 ESP32-C6-MINI-1-N4, U10 INA238, U11 INA238, U12 INA238, U13 INA238, U2 TJA1051T/3, U3 LP5907MFX-3.3, U5 TPS2121RUXR, U612V INA181A2IDBVR, U65V INA181A2IDBVR, U712V TLV7011DBVR, U75V TLV7011DBVR

Commit message: Cleaning up 24 pin schematic
Parts:
- renumbered C612V to C612V1, C65V to C65V1, C712V to C712V1, C75V to C75V1, D_USB to D_USB1, J_SIG to J_SIG1, R_BYP_H to R_BYP_H1, R_BYP_L to R_BYP_L1, U612V to U612V1, U65V to U65V1, U712V to U712V1, U75V to U75V1
Connections:
- net +3V3: no longer C1.2, C10.2, C11.2, C12.2, C13.2, C2.2, C3.2, C4.2, C5.2, C50.2, C6.2, C60.2, C612V1.2, C65V1.2, C7.2, C712V1.2, C75V1.2, C8.2, C9.2, D1.2 (A), D7.2 (A), D_USB1.2 (GND), J1.2 (GND), J1.SH1, J1.SH2, J2.2 (GND), J3.15 (GND), J3.17 (GND), J3.18 (GND), J3.19 (GND), J3.24 (GND), J3.3 (GND), J3.5 (GND), J3.7 (GND), J5.A1 (GND), J5.A12 (GND), J5.B1 (GND), J5.B12 (GND), J5.S1 (SHIELD), J6.10 (GND), J6.12 (GND), J6.14 (GND), J6.15 (GND), J6.16 (GND), J6.4 (GND), J6.7 (GND), J_SIG1.4 (Pin_4), R1.2, R3.2, R50.2, R53.2, R8.2, R9.2, SW1.1, SW2.1, TB6.1, TB7.1, TB8.1, TB9.1, U1.1 (GND), U1.11 (GND), U1.14 (GND), U1.2 (GND), U1.36 (GND), U1.37 (GND), U1.38 (GND), U1.39 (GND), U1.40 (GND), U1.41 (GND), U1.42 (GND), U1.43 (GND), U1.44 (GND), U1.45 (GND), U1.46 (GND), U1.47 (GND), U1.48 (GND), U1.49 (GND), U1.50 (GND), U1.51 (GND), U1.52 (GND), U1.53 (GND), U10.1 (A1), U10.2 (A0), U10.6 (VS), U10.7 (GND), U11.1 (A1), U11.6 (VS), U11.7 (GND), U12.2 (A0), U12.6 (VS), U12.7 (GND), U13.7 (GND), U2.2 (GND), U2.8 (S), U3.2 (GND), U5.12 (GND), U5.3 (CP2), U5.4 (OV2), U5.5 (OV1), U612V1.2 (GND), U612V1.5 (REF), U65V1.2 (GND), U65V1.5 (REF), U712V1.2 (VEE), U75V1.2 (VEE)
- net DETECT: now also R7.2; no longer R7.1
- net DETECT_SENSE: now also R7.1; no longer R7.2
- net PR1: no longer R52.2, R53.1, U5.6 (PR1)
- new net: R52.2, R53.1, U5.6 (PR1)
- new net: U10.7 (GND), U11.6 (VS)
- new net: U11.7 (GND), U12.6 (VS)
- new net GND: C1.2, C10.2, C11.2, C12.2, C13.2, C2.2, C3.2, C4.2, C5.2, C50.2, C6.2, C60.2, C612V1.2, C65V1.2, C7.2, C712V1.2, C75V1.2, C8.2, C9.2, D1.2 (A), D7.2 (A), D_USB1.2 (GND), J1.2 (GND), J1.SH1, J1.SH2, J2.2 (GND), J3.15 (GND), J3.17 (GND), J3.18 (GND), J3.19 (GND), J3.24 (GND), J3.3 (GND), J3.5 (GND), J3.7 (GND), J5.A1 (GND), J5.A12 (GND), J5.B1 (GND), J5.B12 (GND), J5.S1 (SHIELD), J6.10 (GND), J6.12 (GND), J6.14 (GND), J6.15 (GND), J6.16 (GND), J6.4 (GND), J6.7 (GND), J_SIG1.4 (Pin_4), R1.2, R50.2, R53.2, R8.2, R9.2, SW1.1, SW2.1, TB6.1, TB7.1, TB8.1, TB9.1, U1.1 (GND), U1.11 (GND), U1.14 (GND), U1.2 (GND), U1.36 (GND), U1.37 (GND), U1.38 (GND), U1.39 (GND), U1.40 (GND), U1.41 (GND), U1.42 (GND), U1.43 (GND), U1.44 (GND), U1.45 (GND), U1.46 (GND), U1.47 (GND), U1.48 (GND), U1.49 (GND), U1.50 (GND), U1.51 (GND), U1.52 (GND), U1.53 (GND), U10.1 (A1), U10.2 (A0), U11.1 (A1), U12.2 (A0), U12.7 (GND), U13.7 (GND), U2.2 (GND), U2.8 (S), U3.2 (GND), U5.12 (GND), U5.3 (CP2), U5.4 (OV2), U5.5 (OV1), U612V1.2 (GND), U612V1.5 (REF), U65V1.2 (GND), U65V1.5 (REF), U712V1.2 (VEE), U75V1.2 (VEE)
Other:
- moved on the sheet: C1, C2, C3, C4, C5, C50, C6, C60, C612V1, C65V1, C7, C712V1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
