File: modules/atx-24pin-rev3/24pin-module.kicad_pcb (KiCad board)
At the start: 4 copper layers, 82.9 x 79 mm, 49 parts, among them J1 TO-HUB, J2 TO-HUB-PWR, J3 ATX-24 (PSU), J4 ATX-24 (MB), J5 USB_C_Receptacle_USB2.0_16P, SW1 SW_Push, SW2 SW_Push, U1 ESP32-S3-MINI-1-N4R2, U10 INA228, U11 INA228, U12 INA228, U13 INA228, U2 TJA1462A, U3 LP5907MFX-3.3, U4 74LVC1G17, U5 74LVC1G17

Commit message: Tuning up daughterboards and making a new PCB for 24 pin rev3
Parts:
- removed C1, C2: 1uF, cec-Capacitor_SMD:C_0603_1608Metric
- removed C10, C11, C12, C13, C14, C3, C4, C5, C6, C9: 100nF, cec-Capacitor_SMD:C_0402_1005Metric
- removed C15, C7: 10µF, cec-Capacitor_SMD:C_0805_2012Metric
- removed C8: 1µF, cec-Capacitor_SMD:C_0805_2012Metric
- removed D1: D_Schottky, cec-Diode_SMD:D_SMA
- removed D2: LED, cec-LED_SMD:LED_0603_1608Metric
- removed FID1, FID2, FID3: Fiducial_1mm_Mask2mm, cec-Fiducial:Fiducial_1mm_Mask2mm
- removed J1: TO-HUB, cec-Connector_RJ:RJ45_Amphenol_54602-x08_Horizontal
- removed J2: TO-HUB-PWR, cec-Connector_JST:JST_XH_S2B-XH-A_1x02_P2.50mm_Horizontal
- removed J3: ATX-24 (PSU), cec-Connector_Molex:Molex_Mini-Fit_Jr_5569-24A1_2x12_P4.20mm_Horizontal
- removed J4: ATX-24 (MB), cec-Connector_Molex:Molex_Mini-Fit_Jr_5569-24A1_2x12_P4.20mm_Horizontal
- removed J5: USB_C_Receptacle_USB2.0_16P, cec-Connector_USB:USB_C_Receptacle_XKB_U262-16XN-4BVC11
- removed R1: R_ID (OQ-6), cec-Resistor_SMD:R_0402_1005Metric
- removed R10, R7, R9: 1kΩ, cec-Resistor_SMD:R_0402_1005Metric
- removed R2: 10kΩ, cec-Resistor_SMD:R_0402_1005Metric
- removed R3, R4: 2.2kΩ, cec-Resistor_SMD:R_0402_1005Metric
- removed R5, R6: 5.1kΩ, cec-Resistor_SMD:R_0402_1005Metric
- removed RS1, RS2, RS5: R002, cec-Resistor_SMD:R_2512_6332Metric
- removed RS6: R025, cec-Resistor_SMD:R_2512_6332Metric
- removed SW1, SW2: SW_Push, cec-Button_Switch_SMD:Panasonic_EVQPUJ_EVQPUA
- removed U1: ESP32-S3-MINI-1-N4R2, cec-RF_Module:ESP32-S2-MINI-1_NoAntKeepout
- removed U10, U11, U12, U13: INA228, cec-Package_SO:VSSOP-10_3x3mm_P0.5mm
- removed U2: TJA1462A, cec-Package_SO:SOIC-8_3.9x4.9mm_P1.27mm
- removed U3: LP5907MFX-3.3, cec-Package_TO_SOT_SMD:SOT-23-5
- removed U4, U5: 74LVC1G17, cec-Package_TO_SOT_SMD:SOT-23-5
Routing:
- net +5VSB: track 248.8 -> 0.00 mm, vias 7 -> 0
- net +3V3: track 218.8 -> 0.00 mm, vias 10 -> 0
- net GND: track 157.4 -> 0.00 mm, vias 47 -> 0
- net Net-(J3-PWR_OK): track 115.3 -> 0.00 mm, vias 1 -> 0
- net /RAIL5VSB_LO: track 86.2 -> 0.00 mm, vias 4 -> 0
- net Net-(U1-IO8): track 82.2 -> 0.00 mm, vias 4 -> 0
- net Net-(U1-IO9): track 76.7 -> 0.00 mm
- net Net-(J3-PS_ON#): track 66.4 -> 0.00 mm, vias 1 -> 0
- net Net-(J3--12V): track 66.1 -> 0.00 mm
- net /RAIL3V3_LO: track 62.9 -> 0.00 mm, vias 25 -> 0
- net Net-(U1-IO10): track 60.6 -> 0.00 mm, vias 4 -> 0
- net /GPIO0: track 58.0 -> 0.00 mm, vias 2 -> 0
- net /RAIL3V3_HI: track 56.5 -> 0.00 mm, vias 25 -> 0
- net Net-(U1-IO11): track 42.7 -> 0.00 mm, vias 3 -> 0
- net Net-(U1-IO13): track 40.2 -> 0.00 mm, vias 2 -> 0
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- removed copper zone on B.Cu, net /RAIL12V_HI
- removed copper zone on F.Cu, net /RAIL12V_HI
- removed copper zone on B.Cu, net /RAIL12V_LO
- removed copper zone on F.Cu, net /RAIL12V_LO
- removed copper zone on F.Cu, net /RAIL3V3_HI
- removed copper zone on In2.Cu, net /RAIL3V3_HI
- removed copper zone on F.Cu, net /RAIL3V3_LO
- removed copper zone on In2.Cu, net /RAIL3V3_LO
- removed copper zone on F.Cu, net /RAIL5V_HI
- removed copper zone on In2.Cu, net /RAIL5V_HI
- removed copper zone on B.Cu, net /RAIL5V_LO
- removed copper zone on F.Cu, net /RAIL5V_LO
- removed copper zone on In2.Cu, net /RAIL5V_LO
- removed copper zone on In1.Cu, net GND
Other:
- board outline removed

Commit message: Looking through boards and figuring out outlines.
Parts:
- added C1: 1uF, cec-Capacitor_SMD:C_0603_1608Metric, F.Cu at (228.1, 106.9)
- added C10: 100nF, cec-Capacitor_SMD:C_0402_1005Metric, F.Cu at (197.7, 107.5)
- added C11: 100nF, cec-Capacitor_SMD:C_0402_1005Metric, F.Cu at (200.5, 99.6)
- added C12: 100nF, cec-Capacitor_SMD:C_0402_1005Metric, F.Cu at (200.5, 101.6)
- added C13: 100nF, cec-Capacitor_SMD:C_0402_1005Metric, F.Cu at (200.5, 103.5)
- added C2: 1uF, cec-Capacitor_SMD:C_0603_1608Metric, F.Cu at (228.1, 109.4)
- added C3: 100nF, cec-Capacitor_SMD:C_0402_1005Metric, F.Cu at (197.7, 99.6)
- added C4: 100nF, cec-Capacitor_SMD:C_0402_1005Metric, F.Cu at (197.7, 101.6)
- added C5: 100nF, cec-Capacitor_SMD:C_0402_1005Metric, F.Cu at (197.7, 103.5)
- added C50: 2u2, cec-Capacitor_SMD:C_0402_1005Metric, F.Cu at (200.5, 105.5)
- added C6: 10uF, cec-Capacitor_SMD:C_0805_2012Metric, F.Cu at (249.8, 80.4)
- added C60: 100nF, cec-Capacitor_SMD:C_0402_1005Metric, F.Cu at (200.5, 107.5)
- added C612V1: 100nF, cec-Capacitor_SMD:C_0402_1005Metric, F.Cu at (203.4, 99.6)
- added C65V1: 100nF, cec-Capacitor_SMD:C_0402_1005Metric, F.Cu at (203.4, 101.6)
- added C7: 10uF, cec-Capacitor_SMD:C_0805_2012Metric, F.Cu at (249.8, 83.4)
- added C712V1: 100nF, cec-Capacitor_SMD:C_0402_1005Metric, F.Cu at (203.4, 103.5)
- added C75V1: 100nF, cec-Capacitor_SMD:C_0402_1005Metric, F.Cu at (203.4, 105.5)
- added C8: 100nF, cec-Capacitor_SMD:C_0402_1005Metric, F.Cu at (197.7, 105.5)
- added C9: 10uF, cec-Capacitor_SMD:C_0805_2012Metric, F.Cu at (249.8, 86.4)
- added D1: PESD5V0S1BA, cec-Diode_SMD:D_SOD-323, F.Cu at (217.5, 108.2)
- added D2: SS34, cec-Diode_SMD:D_SMA, F.Cu at (200.3, 110.7)
- added D7: PESD5V0S1BA, cec-Diode_SMD:D_SOD-323, F.Cu at (217.5, 111.1)
- added D_USB1: USBLC6-2SC6, cec-Package_TO_SOT_SMD:SOT-23-6, F.Cu at (223.6, 81.3)
- added FB1: 600R@100MHz FB (MPZ2012S601AT000), cec-Capacitor_SMD:C_0805_2012Metric, F.Cu at (249.8, 89.4)
- added FB2: 0R (FB position, populate on EMC evidence), cec-Capacitor_SMD:C_0805_2012Metric, F.Cu at (249.8, 92.4)
- added J1: TO-HUB, cec:RJ45_FTP_Shielded_Horizontal, F.Cu at (192.1, 83.6)
- added J2: TO-HUB-PWR, cec-Connector_JST:JST_XH_S2B-XH-A_1x02_P2.50mm_Horizontal, F.Cu at (245.7, 100.3)
- added J3: ATX-24 PSU, cec-Connector_Molex:Molex_Mini-Fit_Jr_5569-24A1_2x12_P4.20mm_Horizontal, F.Cu at (61.2, 116.8)
- added J5: USB-C 2.0, cec-Connector_USB:USB_C_Receptacle_XKB_U262-16XN-4BVC11, F.Cu at (211.3, 102.0)
- added J6: TO-HUB-STACK, cec-Connector_PinHeader_2.00mm:PinHeader_2x08_P2.00mm_Vertical, F.Cu at (235.6, 80.9)
- added J_SIG1: CEC_CONN_2x5, cec-Connector_PinHeader_2.54mm:PinHeader_2x05_P2.54mm_Vertical, F.Cu at (242.3, 81.6)
- added R1: 2.2kΩ, cec-Resistor_SMD:R_0402_1005Metric, F.Cu at (189.0, 99.6)
- added R2: 10kΩ, cec-Resistor_SMD:R_0402_1005Metric, F.Cu at (189.0, 101.6)
- added R3: 2.2kΩ, cec-Resistor_SMD:R_0402_1005Metric, F.Cu at (189.0, 103.6)
- added R4: 2.2kΩ, cec-Resistor_SMD:R_0402_1005Metric, F.Cu at (189.0, 105.6)
- added R50: 20kΩ, cec-Resistor_SMD:R_0402_1005Metric, F.Cu at (191.9, 103.6)
- added R51: 10kΩ, cec-Resistor_SMD:R_0402_1005Metric, F.Cu at (191.9, 105.6)
- added R52: 100kΩ, cec-Resistor_SMD:R_0402_1005Metric, F.Cu at (191.9, 107.6)
- added R53: 33kΩ, cec-Resistor_SMD:R_0402_1005Metric, F.Cu at (194.8, 99.6)
- added R60: 10kΩ, cec-Resistor_SMD:R_0402_1005Metric, F.Cu at (194.8, 101.6)
- added R7: 100kΩ, cec-Resistor_SMD:R_0402_1005Metric, F.Cu at (189.0, 107.6)
- added R8: 5.1kΩ, cec-Resistor_SMD:R_0402_1005Metric, F.Cu at (191.9, 99.6)
- added R9: 5.1kΩ, cec-Resistor_SMD:R_0402_1005Metric, F.Cu at (191.9, 101.6)
- added RS1: 2mΩ, cec-Resistor_SMD:R_2512_6332Metric, F.Cu at (82.8, 74.8)
- added RS2: 2mΩ, cec-Resistor_SMD:R_2512_6332Metric, F.Cu at (151.5, 125.5)
- added RS3: 2mΩ, cec-Resistor_SMD:R_2512_6332Metric, F.Cu at (186.2, 129.8)
- added RS4: 25mΩ, cec-Resistor_SMD:R_Shunt_Vishay_WSK2512_6332Metric_T1.19mm, F.Cu at (210.4, 109.1)
- added R_BYP_H1: 0Ω, cec-Resistor_SMD:R_0402_1005Metric, F.Cu at (194.8, 103.6)
- added R_BYP_L1: 0Ω, cec-Resistor_SMD:R_0402_1005Metric, F.Cu at (194.8, 105.6)
- added SW1: BOOT, cec-Button_Switch_SMD:TS-1088-AR02016, F.Cu at (229.4, 99.3)
- added SW2: RESET, cec-Button_Switch_SMD:TS-1088-AR02016, F.Cu at (229.4, 103.5)
- added TB1: TE 63969-1, cec-Connector_Blade:TE_63969_FASTON_Receptacle_250_Vertical_THT, F.Cu at (157.4, 56.0)
- added TB10: TE 63969-1, cec-Connector_Blade:TE_63969_FASTON_Receptacle_250_Vertical_THT, F.Cu at (237.4, 74.4)
- added TB2: TE 63969-1, cec-Connector_Blade:TE_63969_FASTON_Receptacle_250_Vertical_THT, F.Cu at (196.0, 74.4)
- added TB3: TE 63969-1, cec-Connector_Blade:TE_63969_FASTON_Receptacle_250_Vertical_THT, F.Cu at (200.6, 74.4)
- added TB4: TE 63969-1, cec-Connector_Blade:TE_63969_FASTON_Receptacle_250_Vertical_THT, F.Cu at (205.9, 74.4)
- added TB5: TE 63969-1, cec-Connector_Blade:TE_63969_FASTON_Receptacle_250_Vertical_THT, F.Cu at (211.1, 74.4)
- added TB6: TE 63969-1, cec-Connector_Blade:TE_63969_FASTON_Receptacle_250_Vertical_THT, F.Cu at (216.4, 74.4)
- added TB7: TE 63969-1, cec-Connector_Blade:TE_63969_FASTON_Receptacle_250_Vertical_THT, F.Cu at (221.6, 74.4)
- added TB8: TE 63969-1, cec-Connector_Blade:TE_63969_FASTON_Receptacle_250_Vertical_THT, F.Cu at (226.9, 74.4)
- added TB9: TE 63969-1, cec-Connector_Blade:TE_63969_FASTON_Receptacle_250_Vertical_THT, F.Cu at (232.1, 74.4)
- added U1: ESP32-C6-MINI-1-N4, cec-RF_Module:ESP32-C6-MINI-1, F.Cu at (213.8, 90.5)
- added U10: INA238, cec-Package_SO:VSSOP-10_3x3mm_P0.5mm, F.Cu at (82.8, 80.2)
- added U11: INA238, cec-Package_SO:VSSOP-10_3x3mm_P0.5mm, F.Cu at (151.5, 130.8)
- added U12: INA238, cec-Package_SO:VSSOP-10_3x3mm_P0.5mm, F.Cu at (186.2, 135.0)
- added U13: INA238, cec-Package_SO:VSSOP-10_3x3mm_P0.5mm, F.Cu at (229.8, 94.9)
- added U2: TJA1051T/3, cec-Package_SO:SOIC-8_3.9x4.9mm_P1.27mm, F.Cu at (244.2, 73.3)
- added U3: LP5907MFX-3.3, cec-Package_TO_SOT_SMD:SOT-23-5, F.Cu at (235.4, 117.2)
- added U5: TPS2121RUXR, cec-Package_DFN_QFN:RUX0012A, F.Cu at (250.2, 71.8)
- added U612V1: INA181A2IDBVR, cec-Package_TO_SOT_SMD:SOT-23-6, F.Cu at (82.9, 70.8)
- added U65V1: INA181A2IDBVR, cec-Package_TO_SOT_SMD:SOT-23-6, F.Cu at (151.5, 121.7)
- added U712V1: TLV7011DBVR, cec-Package_TO_SOT_SMD:SOT-23-5, F.Cu at (88.6, 70.7)
- added U75V1: TLV7011DBVR, cec-Package_TO_SOT_SMD:SOT-23-5, F.Cu at (157.1, 121.5)
Routing:
- net /SENSE3V3_HI: track 0.00 -> 45.5 mm
- net /SENSE12V_LO: track 0.00 -> 11.8 mm
- net +5V_MAIN: track 0.00 -> 10.3 mm
- net /SENSE12V_HI: track 0.00 -> 8.27 mm
- net /SENSE5V_HI: track 0.00 -> 7.76 mm
- added copper zone on F.Cu, net /SENSE12V_HI
- added copper zone on B.Cu, net /SENSE3V3_HI
- added copper zone on B.Cu, net /SENSE5V_HI
