File: beta/pcie-8pin-3port/07-usb-flash.kicad_sch (KiCad schematic)
At the start: 8 parts, among them J5 USB-C 2.0

Commit message: pcie-8pin-3port: USB-ingress TPS2121 mux replaces the D2 SS34 ORing diode (spec v1.6.0 Sec 6.14)
Identical delta and topology to pcie-8pin-2port (docs/usb-ingress-bom-delta-2026-07-24.md
Sec 3.2; see that board's commit for the full rationale) -- the two boards' 07-usb-flash and
01-hub-link leaf sheets share the same coordinates, hierarchical_label mechanics for FB1's
"VBUS_J5" stub, and refdes plan (verified independently against the live pcie-3port file
before running, not assumed from the 2-port board). U4 = TPS2121RUXR: IN1 = RJ-45 VCC feed
after FB2 via a cross-sheet global_label "VCC_RJ45"; IN2 = VBUS behind new polyfuse F1 ahead
of the existing FB1 bead; OUT = +5VSB. OV1/PR1 dividers off IN1; CP2/OV2/GND -> GND; ST left
a genuine no_connect (Output-type pin, avoids the same pin_to_pin ERROR class recorded on
the other two boards). D2 removed entirely; refdes shifted R13->R14.../C41->C42... on the
same pre-existing-part collision as EPS/2-port.

Gates: ERC 122->133, zero new errors (pin_not_driven=1 unchanged pre-existing), pin_to_pin
stays 63, lib_symbol_mismatch +11 (same benign class). Netlist-verified clean on the first
run: +5VSB gains U4.1/U4.8 with no D2 member; /VBUS={C43,C44,C9,D3,D4,FB1.2,U4.2};
/VBUS_J5={F1.1,J5x4}; VCC_RJ45(global)={FB2.2,R15.1,R17.1,U4.7}. BOM regenerated via
scripts/gen-bom-outputs.py --force.

Co-Authored-By: Claude Fable 5 <noreply@anthropic.com>
Parts:
- removed D2: SS34, cec-Diode_SMD:D_SMA, symbol cec-vendor:D_Schottky
- added C42: 2.2uF, cec-Capacitor_SMD:C_0603_1608Metric, symbol cec-vendor:C_Small
- added C43: 100nF, cec-Capacitor_SMD:C_0402_1005Metric, symbol cec-vendor:C_Small
- added C44: 10uF, cec-Capacitor_SMD:C_0805_2012Metric, symbol cec-vendor:C_Small
- added F1: 750mA/16V PTC, cec-Resistor_SMD:R_1206_3216Metric, symbol cec-vendor:R_Small
- added R14, R17: 100kΩ, cec-Resistor_SMD:R_0402_1005Metric, symbol cec-vendor:R_Small
- added R15: 47kΩ, cec-Resistor_SMD:R_0402_1005Metric, symbol cec-vendor:R_Small
- added R16: 10kΩ, cec-Resistor_SMD:R_0402_1005Metric, symbol cec-vendor:R_Small
- added R18: 33kΩ, cec-Resistor_SMD:R_0402_1005Metric, symbol cec-vendor:R_Small
- added U4: TPS2121RUXR, cec-Package_DFN_QFN:RUX0012A, symbol cec-vendor:TPS2121RUXR
Connections:
- net +5VSB: now also U4.1 (OUT), U4.8 (OUT)
- net GND: now also C42.2, C43.2, C44.2, R14.2, R16.2, R18.2, U4.12 (GND), U4.3 (CP2), U4.4 (OV2)
- net VBUS: now also C43.1, C44.1, U4.2 (IN2)
- net VBUS_J5: now also F1.1; no longer FB1.1
- new net U4_ILM: R14.1, U4.10 (ILM)
- new net U4_OV1: R15.2, R16.1, U4.5 (OV1)
- new net U4_PR1: R17.2, R18.1, U4.6 (PR1)
- new net U4_SS: C42.1, U4.11 (SS)
- new net VBUS_F: F1.2, FB1.1
- new net VCC_RJ45: R15.1, R17.1, U4.7 (IN1)
- no-connect marks 2 -> 3
