File: beta/pcie-8pin-3port/07-usb-flash.kicad_sch (KiCad schematic)
At the start: 17 parts, among them J5 USB-C 2.0, U4 TPS2121RUXR

Commit message: Audit BETA electrical and pour pipeline
Parts:
- D4: Manufacturer Nexperia -> HXY MOSFET
Changed lines of the file:
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@@
 		(property "Value" "USB-C 2.0" (at 167.64 74.93 0) (effects (font (size 1.27 1.27))))
 		(property "Footprint" "cec-Connector_USB:USB_C_Receptacle_XKB_U262-16XN-4BVC11" (at 167.64 95.25 0) (effects (font (size 1.27 1.27)) (hide yes)))
-		(property "Datasheet" "" (at 167.64 95.25 0) (effects (font (size 1.27 1.27)) (hide yes)))
+		(property "Datasheet" "https://datasheet.lcsc.com/szlcsc/1811141824_XKB-Enterprise-U262-161N-4BVC11_C319148.pdf" (at 167.64 95.25 0) (effects (font (size 1.27 1.27)) (hide yes)))
 		(property "Manufacturer" "XKB Connection" (at 167.64 95.25 0) (effects (font (size 1.27 1.27)) (hide yes)))
 		(property "MPN" "U262-161N-4BVC11" (at 167.64 95.25 0) (effects (font (size 1.27 1.27)) (hide yes)))
@@
 		(property "Value" "USBLC6-2SC6" (at 97.79 81.026 0) (effects (font (size 1.27 1.27))))
 		(property "Footprint" "cec-Package_TO_SOT_SMD:SOT-23-6" (at 97.79 95.25 0) (effects (font (size 1.27 1.27)) (hide yes)))
-		(property "Datasheet" "" (at 97.79 95.25 0) (effects (font (size 1.27 1.27)) (hide yes)))
+		(property "Datasheet" "https://datasheet.lcsc.com/lcsc/2206231215_UMW-Youtai-Semiconductor-Co---Ltd--USBLC6-2SC6_C2687116.pdf" (at 97.79 95.25 0) (effects (font (size 1.27 1.27)) (hide yes)))
 		(property "Manufacturer" "UMW" (at 97.79 95.25 0) (effects (font (size 1.27 1.27)) (hide yes)))
 		(property "MPN" "USBLC6-2SC6" (at 97.79 95.25 0) (effects (font (size 1.27 1.27)) (hide yes)))
@@
 		(property "Value" "PESD5V0S1BA" (at 129.54 123.19 0) (effects (font (size 1.27 1.27))))
 		(property "Footprint" "cec-Diode_SMD:D_SOD-323" (at 129.54 127 0) (effects (font (size 1.27 1.27)) (hide yes)))
-		(property "Datasheet" "" (at 129.54 127 0) (effects (font (size 1.27 1.27)) (hide yes)))
-		(property "Manufacturer" "Nexperia" (at 129.54 127 0) (effects (font (size 1.27 1.27)) (hide yes)))
+		(property "Datasheet" "https://www.lcsc.com/datasheet/C5261083.pdf" (at 129.54 127 0) (effects (font (size 1.27 1.27)) (hide yes)))
+		(property "Manufacturer" "HXY MOSFET" (at 129.54 127 0) (effects (font (size 1.27 1.27)) (hide yes)))
 		(property "MPN" "PESD5V0S1BA" (at 129.54 127 0) (effects (font (size 1.27 1.27)) (hide yes)))
 		(property "LCSC" "C5261083" (at 129.54 127 0) (effects (font (size 1.27 1.27)) (hide yes)))
@@
 		(property "Value" "TPS2121RUXR" (at 270.51 74.93 0) (effects (font (size 1.27 1.27))))
 		(property "Footprint" "cec-Package_DFN_QFN:RUX0012A" (at 270.51 59.69 0) (effects (font (size 1.27 1.27)) (hide yes)))
-		(property "Datasheet" "" (at 270.51 59.69 0) (effects (font (size 1.27 1.27)) (hide yes)))
+		(property "Datasheet" "https://www.ti.com/lit/ds/symlink/tps2121.pdf" (at 270.51 59.69 0) (effects (font (size 1.27 1.27)) (hide yes)))
 		(property "Manufacturer" "Texas Instruments" (at 270.51 59.69 0) (effects (font (size 1.27 1.27)) (hide yes)))
 		(property "MPN" "TPS2121RUXR" (at 270.51 59.69 0) (effects (font (size 1.27 1.27)) (hide yes)))

Commit message: pipeline: integrate route-aware physical design flow
Generalize critical-first placement and routing, future-congestion and power-authority planning, route provenance, process watchdogs, fab/thermal validation, dashboard review, and XFCN integration. Add the supporting board contracts, component libraries, documentation, and regression coverage.
Parts:
- added C45: 10uF, cec-Capacitor_SMD:C_0805_2012Metric, symbol cec-vendor:C_Small
- R15: value 47kΩ -> 43.2kΩ; LCSC C25792 -> C25894; MPN 0402WGF4702TCE -> 0402WGF4322TCE; Note U4 OV1 divider top (IN1 side). -> U4 OV1 top: 43.2k/10k gives 5.639V nominal, 5.287..5.948V a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
Connections:
- net GND: now also C45.2
- net VCC_RJ45: now also C45.1
Changed lines of the file:
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@@
 		(fields_autoplaced yes)
 		(property "Reference" "R15" (at 299.72 44.45 0) (effects (font (size 1.27 1.27))))
-		(property "Value" "47kΩ" (at 299.72 74.93 0) (effects (font (size 1.27 1.27))))
+		(property "Value" "43.2kΩ" (at 299.72 74.93 0) (effects (font (size 1.27 1.27))))
 		(property "Footprint" "cec-Resistor_SMD:R_0402_1005Metric" (at 299.72 59.69 0) (effects (font (size 1.27 1.27)) (hide yes)))
-		(property "Datasheet" "" (at 299.72 59.69 0) (effects (font (size 1.27 1.27)) (hide yes)))
+		(property "Datasheet" "https://www.lcsc.com/product-detail/C25894.html" (at 299.72 59.69 0) (effects (font (size 1.27 1.27)) (hide yes)))
 		(property "Manufacturer" "UNI-ROYAL" (at 299.72 59.69 0) (effects (font (size 1.27 1.27)) (hide yes)))
-		(property "MPN" "0402WGF4702TCE" (at 299.72 59.69 0) (effects (font (size 1.27 1.27)) (hide yes)))
-		(property "LCSC" "C25792" (at 299.72 59.69 0) (effects (font (size 1.27 1.27)) (hide yes)))
-		(property "Note" "U4 OV1 divider top (IN1 side)." (at 299.72 59.69 0) (effects (font (size 1.27 1.27)) (hide yes)))
+		(property "MPN" "0402WGF4322TCE" (at 299.72 59.69 0) (effects (font (size 1.27 1.27)) (hide yes)))
+		(property "LCSC" "C25894" (at 299.72 59.69 0) (effects (font (size 1.27 1.27)) (hide yes)))
+		(property "Note" "U4 OV1 top: 43.2k/10k gives 5.639V nominal, 5.287..5.948V at 1%/VREF extremes, below the 6.0V regulator absolute maximum." (at 299.72 59.69 0) (effects (font (size 1.27 1.27)) (hide yes)))
 		(pin "1")
 		(pin "2")
@@
 			)
 		)
+	)
+	(symbol
+		(lib_id "cec-vendor:C_Small")
+		(at 229.87 105.41 0)
+		(unit 1)
+		(exclude_from_sim no)
+		(in_bom yes)
+		(on_board yes)
+		(dnp no)
+		(fields_autoplaced yes)
+		(property "Reference" "C45" (at 229.87 90.17 0) (effects (font (size 1.27 1.27))))
+		(property "Value" "10uF" (at 229.87 120.65 0) (effects (font (size 1.27 1.27))))
+		(property "Footprint" "cec-Capacitor_SMD:C_0805_2012Metric" (at 229.87 105.41 0) (effects (font (size 1.27 1.27)) (hide yes)))
+		(property "Datasheet" "https://product.samsungsem.com/mlcc/CL21A106KAYNNN.do" (at 229.87 105.41 0) (effects (font (size 1.27 1.27)) (hide yes)))
+		(property "Manufacturer" "Samsung" (at 229.87 105.41 0) (effects (font (size 1.27 1.27)) (hide yes)))
+		(property "MPN" "CL21A106KAYNNNE" (at 229.87 105.41 0) (effects (font (size 1.27 1.27)) (hide yes)))
+		(property "LCSC" "C15850" (at 229.87 105.41 0) (effects (font (size 1.27 1.27)) (hide yes)))
+		(property "Note" "U4 OUT (VCC_RJ45) local X5R bypass; place directly at OUT and GND." (at 229.87 105.41 0) (effects (font (size 1.27 1.27)) (hide yes)))
+		(pin "1")
+		(pin "2")
+		(instances
+			(project "pcie8pin-3port-module"
+				(path "/a8ecf94e-f41a-4523-8cf1-1d72f47f3e7e/8adba108-789d-4153-ad59-e74c8138b4d8" (reference "C45") (unit 1))
+			)
+		)
+	)
+	(wire (pts (xy 229.87 102.87) (xy 229.87 99.06))
+		(stroke (width 0) (type default)))
+	(global_label "VCC_RJ45"
+		(shape passive)
+		(at 229.87 99.06 0)
+		(fields_autoplaced yes)
+		(effects (font (size 1.27 1.27)) (justify left bottom))
+		(property "Intersheetrefs" "${INTERSHEET_REFS}"
+			(at 229.87 99.06 0)
+			(effects (font (size 1.27 1.27)) (hide yes))
+		)
+	)
+	(wire (pts (xy 229.87 107.95) (xy 229.87 111.76))
+		(stroke (width 0) (type default)))
+	(symbol
+		(lib_id "cec-power:GND")
+		(at 229.87 111.76 0)
+		(unit 1)
+		(exclude_from_sim no)
+		(in_bom yes)
+		(on_board yes)
+		(dnp no)
+		(property "Reference" "#PWR7113" (at 229.87 109.22 0) (effects (font (size 1.27 1.27)) (hide yes)))
+		(property "Value" "GND" (at 229.87 115.57 0) (effects (font (size 1.27 1.27))))
+		(pin "1")
+		(instances
+			(project "pcie8pin-3port-module"
+				(path "/a8ecf94e-f41a-4523-8cf1-1d72f47f3e7e/8adba108-789d-4153-ad59-e74c8138b4d8" (reference "#PWR7113") (unit 1))
+			)
+		)
