File: beta/pcie-8pin-3port/01-hub-link.kicad_sch (KiCad schematic)
At the start: 6 parts, among them J1 TO-HUB

Commit message: Audit BETA electrical and pour pipeline
Parts:
- D1: Manufacturer Nexperia -> HXY MOSFET
Changed lines of the file:
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@@
 		(property "Value" "TO-HUB" (at 133.35 77.47 0) (effects (font (size 1.27 1.27))))
 		(property "Footprint" "cec:RJ45_FTP_Shielded_Horizontal" (at 133.35 90.17 0) (effects (font (size 1.27 1.27)) (hide yes)))
-		(property "Datasheet" "" (at 133.35 90.17 0) (effects (font (size 1.27 1.27)) (hide yes)))
+		(property "Datasheet" "https://www.lcsc.com/datasheet/C2683360.pdf" (at 133.35 90.17 0) (effects (font (size 1.27 1.27)) (hide yes)))
 		(property "Manufacturer" "Kinghelm" (at 133.35 90.17 0) (effects (font (size 1.27 1.27)) (hide yes)))
 		(property "MPN" "KH-RJ45-58-8P8C" (at 133.35 90.17 0) (effects (font (size 1.27 1.27)) (hide yes)))
@@
 		(property "Value" "PESD5V0S1BA" (at 177.8 54.61 0) (effects (font (size 1.27 1.27))))
 		(property "Footprint" "cec-Diode_SMD:D_SOD-323" (at 177.8 58.42 0) (effects (font (size 1.27 1.27)) (hide yes)))
-		(property "Datasheet" "" (at 177.8 58.42 0) (effects (font (size 1.27 1.27)) (hide yes)))
-		(property "Manufacturer" "Nexperia" (at 177.8 58.42 0) (effects (font (size 1.27 1.27)) (hide yes)))
+		(property "Datasheet" "https://www.lcsc.com/datasheet/C5261083.pdf" (at 177.8 58.42 0) (effects (font (size 1.27 1.27)) (hide yes)))
+		(property "Manufacturer" "HXY MOSFET" (at 177.8 58.42 0) (effects (font (size 1.27 1.27)) (hide yes)))
 		(property "MPN" "PESD5V0S1BA" (at 177.8 58.42 0) (effects (font (size 1.27 1.27)) (hide yes)))
 		(property "LCSC" "C5261083" (at 177.8 58.42 0) (effects (font (size 1.27 1.27)) (hide yes)))
