File: beta/hub-standard-rev2/hub-standard-rev2.kicad_sch (KiCad schematic)
At the start: 103 parts, among them J2 PORT1, J3 PORT2, J4 PORT3, J5 PORT4, J6C TO-24PIN-STACK-COMMS, J6D TO-24PIN-STACK-ID, J6P TO-24PIN-STACK-PWR, U1 ESP32-S3-WROOM-1, U10 TPS563201DDCR, U2 TJA1051T/3, U3 LP5907MFX-3.3, U4 TPS3839K33, U5 TPS2121RUXR, U6 SN74AHCT1G08, U7 TPS2121RUXR, U8 TLV7011DBVR, U9 TPS61040DBVR

Commit message: hub-standard-rev2: THIRD TPS2121 cascade stage for J_KVM (spec Sec 2.9 v1.6.0)
docs/usb-ingress-bom-delta-2026-07-24.md Sec 3.5: J_KVM pin 1 (the NanoKVM aux header's
5V line) was a RAW +5VSB power-symbol tap before this splice -- exactly the hazard the
spec's v1.6.0 Sec 2.9 entry describes (a powered Hub could back-drive the NanoKVM's own
USB port; a PC-USB-powered NanoKVM faced the whole Hub 4700uF + module 5VSB tree with
nothing in series; even the intended wall-wart forensic path only worked by back-driving
U7's own OUT). Adds U11 as a third cascade stage, making KVM the lowest-priority input:
MAIN_5V (U7.IN1) > 5VSB/USB (U5 -> U7.IN2, now via U11) > wall-wart/KVM (U11.IN2).

U11.IN1 (pin 7) = /PSU_5V, U5's EXISTING output net -- U11 becomes one more consumer, U5
itself untouched. U11.IN2 (pin 2) = new /KVM_5V_IN, fed from J_KVM.pin1 through new
polyfuse F5 (1.1A hold, defense layer 2). U11.OUT (1,8) = new /PSU_5V_KVM, which REPLACES
U7.pin2's (IN2) AND U7.pin3's (CP2) existing "/PSU_5V" tie -- both pins shared that label
today (U7's own as-built style hard-ties CP2 to IN2, verified live at each pin's own
coordinate), so both move together. This is the detail the doc's own text names only for
IN2; leaving CP2 on the old net would have shorted U11's whole OUT stage back around U7's
own mux onto U5's raw output -- fixed as the as-built pattern requires, not silently
invented, and called out explicitly in the script's own header.

Strap style: "mirror the as-built U5/U7 strap style" per the doc, verified against the
live U5/U7 wiring (not the per-module package's stricter datasheet-default posture) --
CP2 hard-tied to IN2's own net, PR1 hard-tied to IN1's own net, OV1/OV2 -> GND (no
divider), ST left a genuine no_connect. R_ILIM3 (27k, mirrors R_ILIM1/R_ILIM2) and C_SS3
(2.2uF, mirrors C_SS1/C_SS2) match the existing stages' own values/MPNs exactly (verified
against R_ILIM1's own BOM properties before writing, not re-derived blind).

SCOPE NOTE: a mid-task message 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
Parts:
- added C22: 100nF, cec-Capacitor_SMD:C_0402_1005Metric, symbol cec-vendor:C_Small
- added C23: 10uF, cec-Capacitor_SMD:C_0603_1608Metric, symbol cec-vendor:C_Small
- added C_SS3: 2.2uF, cec-Capacitor_SMD:C_0603_1608Metric, symbol cec-vendor:C_Small
- added F5: 1.1A/16V PTC, cec-Resistor_SMD:R_1206_3216Metric, symbol cec-vendor:R_Small
- added R_ILIM3: 27kΩ, cec-Resistor_SMD:R_0402_1005Metric, symbol cec-vendor:R_Small
- added U11: TPS2121RUXR, cec-Package_DFN_QFN:RUX0012A, symbol cec-vendor:TPS2121RUXR
Connections:
- net +5VSB: no longer J_KVM.1 (+5VSB)
- net GND: now also C22.2, C23.2, C_SS3.1, R_ILIM3.2, U11.12 (GND), U11.4 (OV2), U11.5 (OV1)
- net PSU_5V: now also U11.6 (PR1), U11.7 (IN1); no longer U7.2 (IN2), U7.3 (CP2)
- new net KVM_5V_IN: C22.1, C23.1, F5.2, U11.2 (IN2), U11.3 (CP2)
- new net KVM_5V_RAW: F5.1, J_KVM.1 (+5VSB)
- new net PSU_5V_KVM: U11.1 (OUT), U11.8 (OUT), U7.2 (IN2), U7.3 (CP2)
- new net U11_ILM: R_ILIM3.1, U11.10 (ILM)
- new net U11_SS: C_SS3.2, U11.11 (SS)
- no-connect marks 49 -> 50

Commit message: hub-standard-rev2: OV1 dividers on every TPS2121 stage (U5, U7, U11) -- owner ruling 2026-07-24
Owner sign-off landed after this worktree's initial merge point and was independently
verified before acting on it (fetched origin/claude/pipeline-pass-2, confirmed both cited
commits are real, reachable, nathanfraske-bot-authored, and contain the exact claimed
text -- not taken on the citation alone):
  - docs/owner-queue.md commit 8c8ca46f: "Finding 3 SIGNED OFF: hub OV dividers on every
    TPS2121 stage (U5/U7 + the new KVM stage), same 47k/10k ~6.04V posture as the module
    package -- LUMPED into the running schematic pass."
  - commit 9c6083ae / docs/spice-backfeed-verify-2026-07-24.md marginal (F): the TPS2121's
    OV response time is UNDOCUMENTED, and a real 0.8-7.4us over-6.5V-abs-max excursion on
    the LP5907 was measured under a fast cross-rail fault in SPICE -- an OV1 pin hard-
    grounded (the as-built state on all three stages) gives that protection path nothing to
    trigger on, so a correctly-tuned divider on every stage is the mitigation.

Verified live before touching anything (per the instruction: confirm each stage's OV1 pin
isn't committed to a conflicting function first) -- all three were genuinely simple GND
power-symbol ties, nothing else on the node: U5.pin5 at (424.18,105.41), U7.pin5 at
(140.97,361.95), U11.pin5 at (701.04,52.07) [my own build, which mirrored the as-built
hard-GND style per the ORIGINAL delta doc instruction that predates this ruling]. No
conflicts found; all three converted cleanly.

Each stage's divider taps its OWN IN1 net (same "OV1 off IN1" posture as every module's own
mux, spec Sec 6.14): U5 (IN1=/5VSB_RAW) -> R33 (47k) / R34 (10k); U7 (IN1=/MAIN_5V_RAW) ->
R35 (47k) / R36 (10k); U11 (IN1=/PSU_5V) -> R37 (47k) / R38 (10k). Same LCSC parts as every
module divider (C25792/C25744). All three IN1 nets are plain same-sheet local labels on
this flat board (verified: zero power-symbol instances for any of the three names)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
Parts:
- added R33, R35, R37: 47kΩ, cec-Resistor_SMD:R_0402_1005Metric, symbol cec-vendor:R_Small
- added R34, R36, R38: 10kΩ, cec-Resistor_SMD:R_0402_1005Metric, symbol cec-vendor:R_Small
Connections:
- net 5VSB_RAW: now also R33.1
- net GND: now also R34.2, R36.2, R38.2; no longer U11.5 (OV1), U5.5 (OV1), U7.5 (OV1)
- net MAIN_5V_RAW: now also R35.1
- net PSU_5V: now also R37.1
- new net U11_OV1: R37.2, R38.1, U11.5 (OV1)
- new net U5_OV1: R33.2, R34.1, U5.5 (OV1)
- new net U7_OV1: R35.2, R36.1, U7.5 (OV1)
