File: beta/hub-standard-rev2/hub-standard-rev2.kicad_sch (KiCad schematic)
At the start: 115 parts, among them J2 PORT1, J3 PORT2, J4 PORT3, J5 PORT4, J6C TO-24PIN-STACK-COMMS, J6D TO-24PIN-STACK-ID, J6P TO-24PIN-STACK-PWR, U1 ESP32-S3-WROOM-1, U10 TPS563201DDCR, U11 TPS2121RUXR, U2 TJA1051T/3, U3 LP5907MFX-3.3, U4 TPS3839K33, U5 TPS2121RUXR, U6 SN74AHCT1G08, U7 TPS2121RUXR, U8 TLV7011DBVR, U9 TPS61040DBVR

Commit message: Audit BETA electrical and pour pipeline
Parts:
- C23: MPN CL21A106KAYNNNE -> CL10A106MA8NRNC
- D2, D3, D4, D5, D7: Manufacturer Nexperia -> HXY MOSFET
- D8, D9: Manufacturer generic (LCSC pick) -> MDD (Microdiode Semiconductor)
- J6C: Note Segmented mezz per docs/mezz-structural-segments-2026-07-22.md Appendix A (comms segment). STREAM_P/STREAM_N (pins 4/6) intentionally unconnected -- Standard-tier hub carries no RS-485 pair; forward-compat provision only, matches the 24-pin side's unconnected STREAM pads. -> Segmented mezz per docs/mezz-structural-segments-2026-07-22.md Appendix A (comms segment), fitted per docs/decisions/owner-session-2026-08-01.md. STREAM_P/STREAM_N (pins 4/6) are intentionally unconnected on both Standard-tier boards. Exact mating header/socket MPN and stack height remain owner selections.; now fitted
- J6D: Note Segmented mezz per docs/mezz-structural-segments-2026-07-22.md Appendix A (ID segment). RSVD (pin 3) intentionally unconnected -- reserved spare, no net on this board. DETECT ties to /DETECT1 (hub port-1 detect line; role match is what mates, not the literal name). -> Segmented mezz per docs/mezz-structural-segments-2026-07-22.md Appendix A (ID segment), fitted per docs/decisions/owner-session-2026-08-01.md. RSVD (pin 3) is intentionally unconnected. DETECT ties to /DETECT1. Exact mating header/socket MPN and stack height remain owner selections.; now fitted
- J6P: Note Segmented mezz per docs/mezz-structural-segments-2026-07-22.md Appendix A (power segment); supersedes the 2026-07-15 column-paired 2x08 map (flip-invariance premise retired by the 2026-07-19 no-flip ruling). THT + DNP -- facing/assembly per the stack doc. -> Segmented mezz per docs/mezz-structural-segments-2026-07-22.md Appendix A (power segment); supersedes the 2026-07-15 column-paired 2x08 map. Fitted per docs/decisions/owner-session-2026-08-01.md. Exact mating header/socket MPN and stack height remain owner selections.; now fitted
- SW_BOOT, SW_RESET: Manufacturer XKB -> XUNPU
- U1: Manufacturer Espressif -> Espressif Systems
- U2: MPN TJA1051T/3 -> TJA1051T/3/1J; Manufacturer NXP -> NXP Semiconductors
Connections:
- net GND: now also U11.3 (CP2), U5.3 (CP2), U7.3 (CP2)
- net KVM_5V_IN: no longer U11.3 (CP2)
- net PSU_5V_KVM: no longer U7.3 (CP2)
- net USB_VBUS: no longer U5.3 (CP2)

Commit message: Audit BETA power designs and harden PCB pipeline
Parts:
- removed C1: 4700uF, cec-Capacitor_SMD:CP_Elec_16x17.5, symbol cec-vendor:C_Small
- removed C10, C2, C3, C9: 1uF, cec-Capacitor_SMD:C_0603_1608Metric, symbol cec-vendor:C_Small
- removed C11, C23: 10uF, cec-Capacitor_SMD:C_0603_1608Metric, symbol cec-vendor:C_Small
- removed C12: 10nF, cec-Capacitor_SMD:C_0402_1005Metric, symbol cec-vendor:C_Small
- removed C13: 100nF, cec-Capacitor_SMD:C_0603_1608Metric, symbol cec-vendor:C_Small
- removed C14, C15, C16, C17, C18, C19, C20, C21, C22, C4, C5, C6, C8: 100nF, cec-Capacitor_SMD:C_0402_1005Metric, symbol cec-vendor:C_Small
- removed C7: 4n7, cec-Capacitor_SMD:C_0402_1005Metric, symbol cec-vendor:C_Small
- removed C_SS1, C_SS2, C_SS3: 2.2uF, cec-Capacitor_SMD:C_0603_1608Metric, symbol cec-vendor:C_Small
- removed C_bulk1: 470uF, cec-Capacitor_SMD:CP_Elec_6.3x7.7, symbol cec-vendor:C_Small
- removed D1: SS14, cec-Diode_SMD:D_SMA, symbol cec-vendor:SB120
- removed D2, D3, D4, D5, D7: PESD5V0S1BA, cec-Diode_SMD:D_SOD-323, symbol cec-vendor:PESD5V0S1UL
- removed D6: USBLC6-2SC6, cec-Package_TO_SOT_SMD:SOT-23-6, symbol cec-vendor:USBLC6-2SC6
- removed D8, D9: SMAJ5.0A, cec-Diode_SMD:D_SMA, symbol cec-vendor:PESD5V0S1UL
- removed DL1, DL2, DL3, DL4, DL5, DL6, DL7: SK6812MINI-E, cec-LED_SMD:LED_SK6812MINI_PLCC4_3.5x3.5mm_P1.75mm, symbol cec-vendor:SK6812MINI
- removed F1, F2, F3, F4: PTC 500mA, cec-Resistor_SMD:R_0805_2012Metric, symbol cec-vendor:R_Small
- removed F5: 1.1A/16V PTC, cec-Resistor_SMD:R_1206_3216Metric, symbol cec-vendor:R_Small
- removed J2: PORT1, cec:RJ45_FTP_Shielded_Horizontal, symbol cec:CEC_RJ45_8P8C_FTP
- removed J3: PORT2, cec:RJ45_FTP_Shielded_Horizontal, symbol cec:CEC_RJ45_8P8C_FTP
- removed J4: PORT3, cec:RJ45_FTP_Shielded_Horizontal, symbol cec:CEC_RJ45_8P8C_FTP
- removed J5: PORT4, cec:RJ45_FTP_Shielded_Horizontal, symbol cec:CEC_RJ45_8P8C_FTP
- removed J6C: TO-24PIN-STACK-COMMS, cec-Connector_PinHeader_2.54mm:PinHeader_2x04_P2.54mm_Vertical, symbol cec:CEC_CONN_2x4
- removed J6D: TO-24PIN-STACK-ID, cec-Connector_PinHeader_2.54mm:PinHeader_2x02_P2.54mm_Vertical, symbol cec:CEC_CONN_2x2
- removed J6P: TO-24PIN-STACK-PWR, cec-Connector_PinHeader_2.54mm:PinHeader_2x03_P2.54mm_Vertical, symbol cec:CEC_CONN_2x3
- removed J_KVM: CEC_NANOKVM_AUX_5P, cec-Connector_JST:JST_PH_S5B-PH-K-S_1x05_P2.00mm_Horizontal, symbol cec:CEC_NANOKVM_AUX_5P
- removed J_PWR: PWR_IN, cec-Connector_JST:JST_XH_S3B-XH-A_1x03_P2.50mm_Horizontal, symbol cec:CEC_PWR_IN_3P
- removed J_USB: USB-C, cec-Connector_USB:USB_C_Receptacle_XKB_U262-16XN-4BVC11, symbol cec-vendor:USB_C_Receptacle_USB2.0_16P
- removed L2: TBD (rung-3 bench), cec-Inductor_SMD:L_0603_1608Metric, symbol cec-vendor:L_Small
- removed R10, R9: 5.1kΩ, cec-Resistor_SMD:R_0402_1005Metric, symbol cec-vendor:R_Small
- removed R11, R16, R18, R2, R22, R24, R25, R34, R36, R38, R5, R6, R7, R8: 10kΩ, cec-Resistor_SMD:R_0402_1005Metric, symbol cec-vendor:R_Small
- removed R12, R15, R17, R21, R23, R33, R35, R37: 47kΩ, cec-Resistor_SMD:R_0402_1005Metric, symbol cec-vendor:R_Small
- removed R13, R_ILIM1, R_ILIM2, R_ILIM3: 27kΩ, cec-Resistor_SMD:R_0402_1005Metric, symbol cec-vendor:R_Small
- removed R14: 330Ω, cec-Resistor_SMD:R_0402_1005Metric, symbol cec-vendor:R_Small
- removed R19, R20: 33Ω, cec-Resistor_SMD:R_0402_1005Metric, symbol cec-vendor:R_Small
- removed R26: 34.0kOhm, cec-Resistor_SMD:R_0402_1005Metric, symbol cec-vendor:R_Small
- removed R27: 10.0kOhm, cec-Resistor_SMD:R_0402_1005Metric, symbol cec-vendor:R_Small
- removed R28, R31: 1MOhm, cec-Resistor_SMD:R_0402_1005Metric, symbol cec-vendor:R_Small
- removed R29, R30: 100kOhm, cec-Resistor_SMD:R_0402_1005Metric, symbol cec-vendor:R_Small
- removed R3, R4: 60.4, cec-Resistor_SMD:R_0402_1005Metric, symbol cec-vendor:R_Small
- removed R32: 120kOhm, cec-Resistor_SMD:R_0402_1005Metric, symbol cec-vendor:R_Small
- removed RJ_BUCK, RJ_HOLD: 0R (jumper), cec-Resistor_SMD:R_0402_1005Metric, symbol cec-vendor:R_Small
- removed SW_BOOT: SW_BOOT, cec-Button_Switch_SMD:TS-1088-AR02016, symbol cec-vendor:SW_Push
- removed SW_RESET: SW_RST, cec-Button_Switch_SMD:TS-1088-AR02016, symbol cec-vendor:SW_Push
- removed TH1: NTC 10k, cec-Resistor_SMD:NTC_0402_1005Metric, symbol cec-vendor:Thermistor_NTC
- removed U1: ESP32-S3-WROOM-1, cec-RF_Module:ESP32-S3-WROOM-1_NoAntKeepout, symbol cec-vendor:ESP32-S3-WROOM-1
- removed U10: TPS563201DDCR, cec-Package_TO_SOT_SMD:SOT-23-6, symbol cec-vendor:TPS563201DDCR
- removed U11, U5, U7: TPS2121RUXR, cec-Package_DFN_QFN:RUX0012A, symbol cec-vendor:TPS2121RUXR
- removed U2: TJA1051T/3, cec-Package_SO:SOIC-8_3.9x4.9mm_P1.27mm, symbol cec-vendor:TJA1051T-3
- removed U3: LP5907MFX-3.3, cec-Package_TO_SOT_SMD:SOT-23-5, symbol cec-vendor:LP5907MFX-1.2
- removed U4: TPS3839K33, cec-Package_TO_SOT_SMD:SOT-23, symbol cec-vendor:TPS3839DBZ
- removed U6: SN74AHCT1G08, cec-Package_TO_SOT_SMD:SOT-23-5, symbol cec-vendor:SN74AHCT1G08
- removed U8: TLV7011DBVR, cec-Package_TO_SOT_SMD:SOT-23-5, symbol cec-vendor:TLV7011DBVR
- removed U9: TPS61040DBVR, cec-Package_TO_SOT_SMD:SOT-23-5, symbol cec-vendor:TPS61040DBVR
Connections:
- no-connect marks 50 -> 0
Other:
- added sheet CAN + FOUR MODULE PORTS + STACK (04-can-module-ports.kicad_sch)
- added sheet HOLD-UP + 3V3 REGULATOR (02-holdup-3v3.kicad_sch)
- added sheet KVM AUXILIARY + RAIL SENSING (05-kvm-aux-sensors.kicad_sch)
- added sheet MCU + USB SERVICE PORT (03-mcu-usb.kicad_sch)
- added sheet POWER INPUT + SOURCE SELECTION (01-power-input-selection.kicad_sch)
- added sheet STATUS LED CHAIN (06-status-leds.kicad_sch)
- note removed: "BETA-1 (2026-07-03): A4 power-in consolidation, W12 5V-drop comparator (persist-on-fault), H2 rung-3 hold-up DNP provisions (boost+buck, position-only -- see beta-lock-register.md H1/H2 and docs/standard-tier-review/beta-splices/hub-standard.md)"

Commit message: Rework BETA power rails and schematic composition
Other:
- sheet CAN + FOUR MODULE PORTS + STACK ports: added none; removed CAN_H, CAN_L, CAN_MID, VCC_P1, VCC_P2, VCC_P3, VCC_P4
- sheet HOLD-UP + 3V3 REGULATOR ports: added none; removed +5V_HOLD, +HOLD_BOOST, BOOST_EN, BOOST_FB, BUCK_EN, BUCK_FB_3V3, BUCK_SW, BUCK_SW_3V3, COMP_THRESH, HOLD_BUCK_OUT, LOGIC_REG_IN
- sheet KVM AUXILIARY + RAIL SENSING ports: added none; removed AUX_RXC, AUX_TXC, KVM_3V3_REF, KVM_5V_RAW
- sheet MCU + USB SERVICE PORT ports: added none; removed EN, GPIO0, USB_CC1, USB_CC2, USB_DM, USB_DP
- sheet POWER INPUT + SOURCE SELECTION ports: added none; removed PSU_5V, PSU_5V_KVM, U11_ILM, U11_OV1, U11_SS, U5_OV1, U7_ILM, U7_OV1, U7_SS
- sheet STATUS LED CHAIN ports: added none; removed LED_DATA_BUF, LED_DATA_DIN
