File: beta/hub-standard-rev2/01-power-input-selection.kicad_sch (KiCad schematic)
At the start: 28 parts, among them U11 TPS2121RUXR, U5 TPS2121RUXR, U7 TPS2121RUXR

Commit message: Rework BETA power rails and schematic composition
Other:
- note added: "CURRENT LIMIT + OVP SETPOINTS"
- note added: "LOCAL RESERVOIRS + BYPASS"
- note added: "SOURCE MUX DEVICES"

Commit message: pipeline: integrate route-aware physical design flow
Generalize critical-first placement and routing, future-congestion and power-authority planning, route provenance, process watchdogs, fab/thermal validation, dashboard review, and XFCN integration. Add the supporting board contracts, component libraries, documentation, and regression coverage.
Parts:
- removed C24, C9: 1uF, cec-Capacitor_SMD:C_0603_1608Metric, symbol cec-vendor:C_Small
- removed C_SS1: 2.2uF, cec-Capacitor_SMD:C_0603_1608Metric, symbol cec-vendor:C_Small
- removed D9: SMAJ5.0A, cec-Diode_SMD:D_SMA, symbol cec-vendor:PESD5V0S1UL
- removed J_PWR: PWR_IN, cec-Connector_JST:JST_XH_S3B-XH-A_1x03_P2.50mm_Horizontal, symbol cec:CEC_PWR_IN_3P
- removed R33: 47kΩ, cec-Resistor_SMD:R_0402_1005Metric, symbol cec-vendor:R_Small
- removed R34: 10kΩ, cec-Resistor_SMD:R_0402_1005Metric, symbol cec-vendor:R_Small
- removed R_ILIM1: 27kΩ, cec-Resistor_SMD:R_0402_1005Metric, symbol cec-vendor:R_Small
- removed U5: TPS2121RUXR, cec-Package_DFN_QFN:RUX0012A, symbol cec-vendor:TPS2121RUXR
- D8: Note Power-entry TVS (owner GO 2026-07-15): the J_PWR feed arriv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 -> Stack-power TVS: J6P receives the consolidated +5V_SYS rail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
- R35: value 47kΩ -> 43.2kΩ; LCSC C25792 -> C25894; MPN 0402WGF4702TCE -> 0402WGF4322TCE; Note U7 OV1 divider top (MAIN_5V_RAW side) -- owner ruling 2026-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 -> U7 OV1 divider top (+5V_SYS side): 43.2k/10k gives 5.639V n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
- R37: value 47kΩ -> 43.2kΩ; LCSC C25792 -> C25894; MPN 0402WGF4702TCE -> 0402WGF4322TCE; Note U11 OV1 divider top (PSU_5V side) -- owner ruling 2026-07-2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 -> U11 OV1 divider top (USB_VBUS side): 43.2k/10k gives 5.639V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
Connections:
- net PSU_5V is gone; now on net USB_VBUS: C25.1, R37.1, U11.6 (PR1), U11.7 (IN1)
- net PWR_SOURCE_STATUS: now reaches U7.9 (ST)
- net MAIN_5V_RAW renamed +5V_SYS
- no-connect marks 3 -> 1
Other:
- note added: "Two TPS2121 stages: stack +5V_SYS primary, protected USB/KVM backup, OV/current limits and local reservoirs."
- note removed: "Three TPS2121 stages, protected inputs, current limits, OV thresholds and local reservoirs."
