File: beta/argb-standard/04-can.kicad_sch (KiCad schematic)
At the start: 6 parts, among them U2 TJA1051T/3

Commit message: Audit BETA electrical and pour pipeline
Parts:
- U2: MPN TJA1051T/3 -> TJA1051T/3/1J; Manufacturer NXP -> NXP Semiconductors
Changed lines of the file:
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@@
 		(property "Value" "TJA1051T/3" (at 114.3 76.2 0) (effects (font (size 1.27 1.27))))
 		(property "Footprint" "cec-Package_SO:SOIC-8_3.9x4.9mm_P1.27mm" (at 114.3 97.79 0) (effects (font (size 1.27 1.27)) (hide yes)))
-		(property "Datasheet" "" (at 114.3 97.79 0) (effects (font (size 1.27 1.27)) (hide yes)))
-		(property "Manufacturer" "NXP" (at 114.3 97.79 0) (effects (font (size 1.27 1.27)) (hide yes)))
-		(property "MPN" "TJA1051T/3" (at 114.3 97.79 0) (effects (font (size 1.27 1.27)) (hide yes)))
+		(property "Datasheet" "https://www.nxp.com/docs/en/data-sheet/TJA1051.pdf" (at 114.3 97.79 0) (effects (font (size 1.27 1.27)) (hide yes)))
+		(property "Manufacturer" "NXP Semiconductors" (at 114.3 97.79 0) (effects (font (size 1.27 1.27)) (hide yes)))
+		(property "MPN" "TJA1051T/3/1J" (at 114.3 97.79 0) (effects (font (size 1.27 1.27)) (hide yes)))
 		(property "LCSC" "C38695" (at 114.3 97.79 0) (effects (font (size 1.27 1.27)) (hide yes)))
 		(pin "1")
