File: beta/argb-standard/08-status.kicad_sch (KiCad schematic)
At the start: 4 parts, among them U6 SN74AHCT1G08

Commit message: Finalize compact Hub and ATX power-layout audit
Parts:
- DL1: Manufacturer Opsco -> OPSCO Optoelectronics
Changed lines of the file:
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@@
 		(property "Footprint" "cec-LED_SMD:LED_SK6812MINI_PLCC4_3.5x3.5mm_P1.75mm" (at 184.15 115.57 0) (effects (font (size 1.27 1.27)) (hide yes)))
 		(property "Datasheet" "" (at 184.15 115.57 0) (effects (font (size 1.27 1.27)) (hide yes)))
-		(property "Manufacturer" "Opsco" (at 184.15 115.57 0) (effects (font (size 1.27 1.27)) (hide yes)))
+		(property "Manufacturer" "OPSCO Optoelectronics" (at 184.15 115.57 0) (effects (font (size 1.27 1.27)) (hide yes)))
 		(property "MPN" "SK6812MINI-E" (at 184.15 115.57 0) (effects (font (size 1.27 1.27)) (hide yes)))
 		(property "LCSC" "C5149201" (at 184.15 115.57 0) (effects (font (size 1.27 1.27)) (hide yes)))
