File: beta/eps-8pin/06-cable-power.kicad_sch (KiCad schematic)
At the start: 16 parts

Commit message: Audit BETA electrical and pour pipeline
Parts:
- J_IN1, J_IN2: MPN (none) -> 87427-0802; Manufacturer (none) -> Molex
Changed lines of the file:
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@@
 			)
 		)
-		(property "Datasheet" ""
+		(property "Datasheet" "https://www.molex.com/content/dam/molex/molex-dot-com/products/automated/en-us/productspecificationpdf/874/87427/PS-87427-0001-001.pdf"
 			(at 149.86 26.67 0)
 			(hide yes)
@@
 			)
 		)
+		(property "MPN" "87427-0802" (at 0 0 0) (effects (font (size 1.27 1.27)) (hide yes)))
+		(property "Manufacturer" "Molex" (at 0 0 0) (effects (font (size 1.27 1.27)) (hide yes)))
 		(property "Description" ""
 			(at 149.86 26.67 0)
@@
 			)
 		)
-		(property "Datasheet" ""
+		(property "Datasheet" "https://www.molex.com/content/dam/molex/molex-dot-com/products/automated/en-us/productspecificationpdf/874/87427/PS-87427-0001-001.pdf"
 			(at 149.86 83.82 0)
 			(hide yes)
@@
 			)
 		)
+		(property "MPN" "87427-0802" (at 0 0 0) (effects (font (size 1.27 1.27)) (hide yes)))
+		(property "Manufacturer" "Molex" (at 0 0 0) (effects (font (size 1.27 1.27)) (hide yes)))
 		(property "Description" ""
 			(at 149.86 83.82 0)
