File: beta/pcie-8pin-2port/03-ldo.kicad_sch (KiCad schematic)
At the start: 3 parts, among them U3 LP5907MFX-3.3

Commit message: Audit BETA electrical and pour pipeline
Parts:
- C1, C2: MPN CL10B105KO8NNNC -> CL10A105KB8NNNC
- U3: MPN LP5907MFX-3.3 -> LP5907MFX-3.3/NOPB
Changed lines of the file:
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@@
 		(property "Value" "LP5907MFX-3.3" (at 147.32 95.25 0) (effects (font (size 1.27 1.27))))
 		(property "Footprint" "cec-Package_TO_SOT_SMD:SOT-23-5" (at 147.32 102.87 0) (effects (font (size 1.27 1.27)) (hide yes)))
-		(property "Datasheet" "" (at 147.32 102.87 0) (effects (font (size 1.27 1.27)) (hide yes)))
+		(property "Datasheet" "https://www.ti.com/lit/ds/symlink/lp5907.pdf" (at 147.32 102.87 0) (effects (font (size 1.27 1.27)) (hide yes)))
 		(property "Manufacturer" "Texas Instruments" (at 147.32 102.87 0) (effects (font (size 1.27 1.27)) (hide yes)))
-		(property "MPN" "LP5907MFX-3.3" (at 147.32 102.87 0) (effects (font (size 1.27 1.27)) (hide yes)))
+		(property "MPN" "LP5907MFX-3.3/NOPB" (at 147.32 102.87 0) (effects (font (size 1.27 1.27)) (hide yes)))
 		(property "LCSC" "C80670" (at 147.32 102.87 0) (effects (font (size 1.27 1.27)) (hide yes)))
 		(pin "1")
@@
 		(property "Datasheet" "" (at 179.07 87.63 0) (effects (font (size 1.27 1.27)) (hide yes)))
 		(property "Manufacturer" "Samsung" (at 179.07 87.63 0) (effects (font (size 1.27 1.27)) (hide yes)))
-		(property "MPN" "CL10B105KO8NNNC" (at 179.07 87.63 0) (effects (font (size 1.27 1.27)) (hide yes)))
+		(property "MPN" "CL10A105KB8NNNC" (at 179.07 87.63 0) (effects (font (size 1.27 1.27)) (hide yes)))
 		(property "LCSC" "C15849" (at 179.07 87.63 0) (effects (font (size 1.27 1.27)) (hide yes)))
 		(pin "1")
@@
 		(property "Datasheet" "" (at 179.07 118.11 0) (effects (font (size 1.27 1.27)) (hide yes)))
 		(property "Manufacturer" "Samsung" (at 179.07 118.11 0) (effects (font (size 1.27 1.27)) (hide yes)))
-		(property "MPN" "CL10B105KO8NNNC" (at 179.07 118.11 0) (effects (font (size 1.27 1.27)) (hide yes)))
+		(property "MPN" "CL10A105KB8NNNC" (at 179.07 118.11 0) (effects (font (size 1.27 1.27)) (hide yes)))
 		(property "LCSC" "C15849" (at 179.07 118.11 0) (effects (font (size 1.27 1.27)) (hide yes)))
 		(pin "1")
