File: beta/pcie-8pin-2port/02-can.kicad_sch (KiCad schematic)
At the start: 6 parts, among them U2 TJA1051T/3

Commit message: Audit BETA electrical and pour pipeline
Parts:
- U2: MPN TJA1051T/3 -> TJA1051T/3/1J; Manufacturer NXP -> NXP Semiconductors
Changed lines of the file:
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@@
 		(property "Value" "TJA1051T/3" (at 157.48 63.5 0) (effects (font (size 1.27 1.27))))
 		(property "Footprint" "cec-Package_SO:SOIC-8_3.9x4.9mm_P1.27mm" (at 157.48 88.9 0) (effects (font (size 1.27 1.27)) (hide yes)))
-		(property "Datasheet" "" (at 157.48 88.9 0) (effects (font (size 1.27 1.27)) (hide yes)))
-		(property "Manufacturer" "NXP" (at 157.48 88.9 0) (effects (font (size 1.27 1.27)) (hide yes)))
-		(property "MPN" "TJA1051T/3" (at 157.48 88.9 0) (effects (font (size 1.27 1.27)) (hide yes)))
+		(property "Datasheet" "https://www.nxp.com/docs/en/data-sheet/TJA1051.pdf" (at 157.48 88.9 0) (effects (font (size 1.27 1.27)) (hide yes)))
+		(property "Manufacturer" "NXP Semiconductors" (at 157.48 88.9 0) (effects (font (size 1.27 1.27)) (hide yes)))
+		(property "MPN" "TJA1051T/3/1J" (at 157.48 88.9 0) (effects (font (size 1.27 1.27)) (hide yes)))
 		(property "LCSC" "C38695" (at 157.48 88.9 0) (effects (font (size 1.27 1.27)) (hide yes)))
 		(pin "1")

Commit message: pipeline: integrate route-aware physical design flow
Generalize critical-first placement and routing, future-congestion and power-authority planning, route provenance, process watchdogs, fab/thermal validation, dashboard review, and XFCN integration. Add the supporting board contracts, component libraries, documentation, and regression coverage.
Parts:
- FL1: now left out of the parts list
Changed lines of the file:
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@@
 		(unit 1)
 		(exclude_from_sim no)
-		(in_bom yes)
-		(on_board yes)
+		(in_bom no)
+		(on_board no)
 		(dnp yes)
 		(fields_autoplaced yes)

Commit message: pipeline: close current-beta decoupler cells
Connections:
- net +5VSB: now also C8.2
- net GND: no longer C8.2
Changed lines of the file:
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@@
 	)
 	(symbol
-		(lib_id "cec-power:GND")
+		(lib_id "cec-power:+5VSB")
 		(at 201.93 114.3 0)
 		(unit 1)
@@
 		(dnp no)
 		(property "Reference" "#PWR202" (at 201.93 111.76 0) (effects (font (size 1.27 1.27)) (hide yes)))
-		(property "Value" "GND" (at 201.93 119.38 0) (effects (font (size 1.27 1.27))))
+		(property "Value" "+5VSB" (at 201.93 119.38 0) (effects (font (size 1.27 1.27))))
 		(pin "1")
 		(instances
