File: beta/12vhpwr-standard/03-output.kicad_sch (KiCad schematic)
At the start: 1 part, among them J4 12V-2x6 OUT pigtail

Commit message: Audit BETA power designs and harden PCB pipeline
Changed lines of the file:
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@@
 	(wire (pts (xy 140.97 92.71) (xy 137.16 92.71))
-		(stroke (width 0) (type default)))
-	(wire (pts (xy 156.21 95.25) (xy 160.02 95.25))
-		(stroke (width 0) (type default)))
-	(wire (pts (xy 156.21 97.79) (xy 161.29 97.79))
-		(stroke (width 0) (type default)))
-	(wire (pts (xy 156.21 100.33) (xy 162.56 100.33))
 		(stroke (width 0) (type default)))
 	(wire (pts (xy 140.97 107.95) (xy 137.16 107.95))
@@
 	(wire (pts (xy 140.97 110.49) (xy 135.89 110.49))
 		(stroke (width 0) (type default)))
-	(wire (pts (xy 156.21 92.71) (xy 161.29 92.71))
+	(wire (pts (xy 156.21 92.71) (xy 160.02 92.71))
 		(stroke (width 0) (type default)))
 	(wire (pts (xy 137.16 92.71) (xy 113.03 92.71))
@@
 	(symbol
 		(lib_id "cec-power:GND")
-		(at 160.02 95.25 0)
-		(unit 1)
-		(exclude_from_sim no)
-		(in_bom yes)
-		(on_board yes)
-		(dnp no)
-		(property "Reference" "#PWR301" (at 160.02 92.71 0) (effects (font (size 1.27 1.27)) (hide yes)))
-		(property "Value" "GND" (at 160.02 109.22 0) (effects (font (size 1.27 1.27))))
-		(pin "1")
-		(instances
-			(project "12vhpwr-standard-module"
-				(path "/436b24cb-7227-4a56-93c7-4c5d9a5d0058/3c9d5a2e-6b0a-4b6b-9a7a-2f7a7a8a1a03" (reference "#PWR301") (unit 1))
-			)
-		)
-	)
-	(symbol
-		(lib_id "cec-power:GND")
-		(at 161.29 97.79 0)
-		(unit 1)
-		(exclude_from_sim no)
-		(in_bom yes)
-		(on_board yes)
-		(dnp no)
-		(property "Reference" "#PWR302" (at 161.29 95.25 0) (effects (font (size 1.27 1.27)) (hide yes)))
-		(property "Value" "GND" (at 161.29 111.76 0) (effects (font (size 1.27 1.27))))
-		(pin "1")
-		(instances
-			(project "12vhpwr-standard-module"
-				(path "/436b24cb-7227-4a56-93c7-4c5d9a5d0058/3c9d5a2e-6b0a-4b6b-9a7a-2f7a7a8a1a03" (reference "#PWR302") (unit 1))
-			)
-		)
-	)
-	(symbol
-		(lib_id "cec-power:GND")
-		(at 162.56 100.33 0)
-		(unit 1)
-		(exclude_from_sim no)
-		(in_bom yes)
-		(on_board yes)
-		(dnp no)
-		(property "Reference" "#PWR303" (at 162.56 97.79 0) (effects (font (size 1.27 1.27)) (hide yes)))
-		(property "Value" "GND" (at 162.56 106.68 0) (effects (font (size 1.27 1.27))))
-		(pin "1")
-		(instances
-			(project "12vhpwr-standard-module"
-				(path "/436b24cb-7227-4a56-93c7-4c5d9a5d0058/3c9d5a2e-6b0a-4b6b-9a7a-2f7a7a8a1a03" (reference "#PWR303") (unit 1))
-			)
-		)
-	)
-	(symbol
-		(lib_id "cec-power:GND")
 		(at 137.16 107.95 0)
 		(unit 1)
@@
 	(symbol
 		(lib_id "cec-power:GND")
-		(at 161.29 92.71 0)
+		(at 160.02 92.71 0)
 		(unit 1)
 		(exclude_from_sim no)
@@
 		(on_board yes)
 		(dnp no)
-		(property "Reference" "#PWR306" (at 161.29 90.17 0) (effects (font (size 1.27 1.27)) (hide yes)))
-		(property "Value" "GND" (at 161.29 104.14 0) (effects (font (size 1.27 1.27))))
+		(property "Reference" "#PWR306" (at 160.02 90.17 0) (effects (font (size 1.27 1.27)) (hide yes)))
+		(property "Value" "GND" (at 160.02 104.14 0) (effects (font (size 1.27 1.27))))
 		(pin "1")
 		(instances
@@
 		)
 	)
-	(sheet_instances
+		(wire (pts (xy 156.21 92.71) (xy 156.21 95.25))
+		(stroke (width 0) (type default)))
+	(wire (pts (xy 156.21 95.25) (xy 156.21 97.79))
+		(stroke (width 0) (type default)))
+	(wire (pts (xy 156.21 97.79) (xy 156.21 100.33))
+		(stroke (width 0) (type default)))
+(sheet_instances
 		(path "/3c9d5a2e-6b0a-4b6b-9a7a-2f7a7a8a1a03"
 			(page "4")

Commit message: Rework BETA power rails and schematic composition
Changed lines of the file:
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@@
 		(dnp no)
 		(fields_autoplaced yes)
-		(property "Reference" "J4" (at 148.59 86.36 0) (effects (font (size 1.27 1.27))))
-		(property "Value" "12V-2x6 OUT pigtail" (at 148.59 88.9 0) (effects (font (size 1.27 1.27))))
+		(property "Reference" "J4" (at 154.94 86.36 0) (effects (font (size 1.27 1.27)) (justify left)))
+		(property "Value" "12V-2x6 OUT pigtail" (at 154.94 88.9 0) (effects (font (size 1.27 1.27)) (justify left)))
 		(property "Footprint" "cec:CEC_12V2x6_Horizontal" (at 148.59 101.6 0) (effects (font (size 1.27 1.27)) (hide yes)))
 		(property "Datasheet" "" (at 148.59 101.6 0) (effects (font (size 1.27 1.27)) (hide yes)))
