File: beta/eps-8pin-rev3/01-hub-can.kicad_sch (KiCad schematic)
At the start: 7 parts, among them J1 TO-HUB, U2 TJA1051T/3

Commit message: Enforce readable BETA schematic layouts
Changed lines of the file:
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@@
 		(rev "DRAFT")
 		(company "CEC")
-		(comment 1 "Protected DETECT input and the module CAN transceiver at the hub connector.")
+		(comment 1 "Protected DETECT input and the module CAN transceiver at the...")
 	)
 	(text "HUB LINK + CAN"
@@
 		(dnp no)
 		(fields_autoplaced yes)
-		(property "Reference" "J1" (at 74.93 74.93 0) (effects (font (size 1.27 1.27))))
-		(property "Value" "TO-HUB" (at 74.93 77.47 0) (effects (font (size 1.27 1.27))))
+		(property "Reference" "J1" (at 82.55 74.93 0) (effects (font (size 1.27 1.27)) (justify left)))
+		(property "Value" "TO-HUB" (at 82.55 77.47 0) (effects (font (size 1.27 1.27)) (justify left)))
 		(property "Footprint" "cec:RJ45_FTP_Shielded_Horizontal" (at 74.93 90.17 0) (effects (font (size 1.27 1.27)) (hide yes)))
 		(property "Datasheet" "https://www.lcsc.com/datasheet/C2683360.pdf" (at 74.93 90.17 0) (effects (font (size 1.27 1.27)) (hide yes)))
@@
 		(dnp no)
 		(fields_autoplaced yes)
-		(property "Reference" "U2" (at 74.93 114.3 0) (effects (font (size 1.27 1.27))))
-		(property "Value" "TJA1051T/3" (at 74.93 109.22 0) (effects (font (size 1.27 1.27))))
+		(property "Reference" "U2" (at 87.63 118.11 0) (effects (font (size 1.27 1.27)) (justify left)))
+		(property "Value" "TJA1051T/3" (at 87.63 120.65 0) (effects (font (size 1.27 1.27)) (justify left)))
 		(property "Footprint" "cec-Package_SO:SOIC-8_3.9x4.9mm_P1.27mm" (at 74.93 130.81 0) (effects (font (size 1.27 1.27)) (hide yes)))
 		(property "Datasheet" "https://www.nxp.com/docs/en/data-sheet/TJA1051.pdf" (at 74.93 130.81 0) (effects (font (size 1.27 1.27)) (hide yes)))

Commit message: pipeline: integrate route-aware physical design flow
Generalize critical-first placement and routing, future-congestion and power-authority planning, route provenance, process watchdogs, fab/thermal validation, dashboard review, and XFCN integration. Add the supporting board contracts, component libraries, documentation, and regression coverage.
Connections:
- net +5VSB: no longer J1.1 (VCC)
- new net VCC_RJ45: J1.1 (VCC)
Changed lines of the file:
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@@
 	(wire (pts (xy 128.27 128.27) (xy 128.27 124.46))
-		(stroke (width 0) (type default)))
-	(wire (pts (xy 64.77 81.28) (xy 60.96 81.28))
 		(stroke (width 0) (type default)))
 	(wire (pts (xy 74.93 120.65) (xy 74.93 116.84))
@@
 	(symbol
 		(lib_id "cec-power:+5VSB")
-		(at 60.96 81.28 180)
-		(unit 1)
-		(exclude_from_sim no)
-		(in_bom yes)
-		(on_board yes)
-		(dnp no)
-		(property "Reference" "#PWR104" (at 60.96 78.74 0) (effects (font (size 1.27 1.27)) (hide yes)))
-		(property "Value" "+5VSB" (at 60.96 91.44 0) (effects (font (size 1.27 1.27))))
-		(pin "1")
-		(instances
-			(project "eps-8pin-rev3"
-				(path "/ef7f6c4c-2dd9-4559-b472-96b33604786a/ef5c2d96-f002-5929-9940-f7976e9dfcc0" (reference "#PWR104") (unit 1))
-			)
-		)
-	)
-	(symbol
-		(lib_id "cec-power:+5VSB")
 		(at 74.93 116.84 0)
 		(unit 1)
@@
 	(no_connect (at 64.77 91.44))
 	(no_connect (at 64.77 96.52))
+	(wire (pts (xy 64.77 81.28) (xy 60.96 81.28))
+		(stroke (width 0) (type default)))
+	(global_label "VCC_RJ45"
+		(shape passive)
+		(at 60.96 81.28 180)
+		(fields_autoplaced yes)
+		(effects (font (size 1.27 1.27)) (justify right bottom))
+		(property "Intersheetrefs" "${INTERSHEET_REFS}"
+			(at 60.96 81.28 0)
+			(effects (font (size 1.27 1.27)) (hide yes))
+		)
+	)
 	(sheet_instances
 		(path "/ef5c2d96-f002-5929-9940-f7976e9dfcc0"
