File: beta/pcie-8pin-3port/candidate/pcie-8pin-3port-candidate.kicad_pcb (KiCad board)
At the start: 4 copper layers, 103.5 x 59.6 mm, 92 parts, among them J1 TO-HUB, J5 USB-C 2.0, SW1 BOOT, SW2 RESET, U1 ESP32-C6-MINI-1-N4, U10 INA238, U11 INA238, U12 INA238, U2 TJA1051T/3, U20 INA181A2IDBVR, U21 INA181A2IDBVR, U22 INA181A2IDBVR, U3 LP5907MFX-3.3, U30 TLV7011DBVR, U31 TLV7011DBVR, U32 TLV7011DBVR, U4 TPS2121RUXR

Commit message: pipeline: integrate route-aware physical design flow
Generalize critical-first placement and routing, future-congestion and power-authority planning, route provenance, process watchdogs, fab/thermal validation, dashboard review, and XFCN integration. Add the supporting board contracts, component libraries, documentation, and regression coverage.
Parts:
- removed TB12, TB14, TB15, TB16, TB22, TB24, TB25, TB26, TB32, TB34, TB35, TB36: TE 63969-1, cec-Connector_Blade:TE_63969_FASTON_Receptacle_250_Vertical_THT
- added C45: 10uF, C_0805_2012Metric, F.Cu at (57.0, 38.0)
- added R19: 10kΩ, R_0402_1005Metric, F.Cu at (46.1, 32.4)
- C7: value 10uF -> 4.7uF
- R15: value 47kΩ -> 43.2kΩ
- TB11, TB13, TB21, TB23, TB31, TB33: value TE 63969-1 -> TTR32100127-0600; footprint cec-Connector_Blade:TE_63969_FASTON_Receptacle_250_Vertical_THT -> cec-Connector_Screw:XFCN_TTR32100127-0600_THT_M3_60A
- moved TB13 24.0 mm to (29.8, 54.5)
- moved TB23 23.0 mm to (58.8, 54.5)
- moved TB33 22.0 mm to (87.8, 54.5)
- moved J_IN1 6.00 mm to (18.8, 1.80)
- moved J_IN3 6.00 mm to (72.5, 1.80)
- moved TB31 1.57 mm to (73.8, 54.5)
- moved TB11 0.93 mm to (15.8, 54.5)
- moved TB21 0.81 mm to (44.8, 54.5)
Connections:
- H1 pad 1: GND -> (no net)
- H2 pad 1: GND -> (no net)
- H3 pad 1: GND -> (no net)
- U1 pad 22: unconnected-(U1-IO8-Pad22) -> /04-mcu/IO8_STRAP
